File: kicad/om_clip/om_clip.kicad_sch (KiCad schematic)
At the start: 17 parts, among them J2 Conn_01x06_Pin, Q1 NPN, Q2 NPN, U1 LM393

Commit message: added structure and dual input
Connections:
- net MON-A renamed MON_1
- net MON-B renamed MON_2
Changed lines of the file:
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@@
 		)
 	)
-	(label "MON-A"
+	(label "MON_1"
 		(at 153.67 100.33 180)
 		(effects
@@
 		)
 	)
-	(label "MON-A"
+	(label "MON_1"
 		(at 143.51 133.35 0)
 		(effects
@@
 		)
 	)
-	(label "MON-B"
+	(label "MON_2"
 		(at 143.51 135.89 0)
 		(effects
@@
 		)
 	)
-	(label "MON-B"
+	(label "MON_2"
 		(at 134.62 100.33 0)
 		(effects
