File: kicad/om_input/om_input.kicad_sch (KiCad schematic)
At the start: 63 parts, among them J1 XLR3_AudioJack3_Combo_Switch, J2 Conn_01x08_Pin, Q1 PNP, Q2 PNP, SW1 SW_DPDT_x2, SW2 SW_4PDT_x4, U1 TL072, U2 NE5532, U3 NE5532, U4 NE5532, U5 NE5532

Commit message: added structure and dual input
Parts:
- removed J2: Conn_01x08_Pin, symbol Connector:Conn_01x08_Pin
- added C15: 100nF, symbol Device:C
- added C16, C17, C22, C26, C27: 47uF, symbol Device:C_Polarized_US
- added C18: 100pF, symbol Device:C
- added C19, C20, C21: 680pF, symbol Device:C
- added C23: 470uF, symbol Device:C_Polarized_US
- added C24, C28: 12pF, symbol Device:C
- added C25: 15pF, symbol Device:C
- added D10, D11, D12, D8, D9: D, symbol Device:D
- added D7: LED, symbol Device:LED
- added J15: XLR3_AudioJack3_Combo_Switch, symbol Connector_Audio:XLR3_AudioJack3_Combo_Switch
- added J16: Conn_01x11_Pin, symbol Connector:Conn_01x11_Pin
- added Q3, Q4: PNP, symbol Simulation_SPICE:PNP
- added R32: 330, symbol Device:R_US
- added R33, R34: 6k8, symbol Device:R_US
- added R35, R60: 100, symbol Device:R_US
- added R36, R38, R46: 2k2, symbol Device:R_US
- added R37: 1M, symbol Device:R_US
- added R39: 1k3, symbol Device:R_US
- added R40, R41, R58, R59: 22k, symbol Device:R_US
- added R42, R51: 10k, symbol Device:R_US
- added R43, R52: 4k7, symbol Device:R_US
- added R44: 100R, symbol Device:R_US
- added R45, R57: 2k7, symbol Device:R_US
- added R47, R48, R49, R50: 1k, symbol Device:R_US
- added R53, R54, R61, R62: 1k5, symbol Device:R_US
- added R55, R56: 470, symbol Device:R_US
- added RV2: 10k, symbol openmic:R_Potentiometer_US_Dual
- added SW3: SW_DPDT_x2, symbol Switch:SW_DPDT_x2
- added SW4: SW_4PDT_x4, symbol openmic:SW_4PDT_x4
- added U10, U8, U9: NE5532, symbol Amplifier_Operational:NE5532
- R7: value 1k8 -> 2k2
- R8: value 3k9 -> 1k3
Connections:
- net +15V: now also J16.3 (Pin_3), R42.1, R51.1, U10.8 (V+), U8.8 (V+), U9.8 (V+)
- net +48V: now also J16.1 (Pin_1), SW3.3 (C)
- net +5V: now also J16.2 (Pin_2), SW3.6 (C)
- net -15V: now also D11.2 (A), D8.2 (A), J16.4 (Pin_4), R43.2, R52.2, U10.4 (V-), U8.4 (V-), U9.4 (V-)
- net Earth: now also U5.5 (+), C18.1, C20.2, C21.2, D7.1 (K), J15.1, J15.S, J15.SN, J16.5 (Pin_5), R37.1, R38.2, R40.2, R41.2, R49.2, R50.1, R56.2, R60.2, SW3.1 (A), SW3.4 (A), SW4.12 (C), SW4.2 (B), U9.5 (+)
- net at U5.6 (-): now also C28.1, R61.2, R62.1
- net SIG_2-: now reaches U5.7
- net SIG_2-: now also C28.2, J16.10 (Pin_10), R62.2
- net at U1.5 (+): now also C15.2, C18.2, R37.2
- net at U1.6 (-): now also R38.1, R39.2
- net at U1.7: now also C22.1, R39.1
- net MON renamed MON_1
- net MON_1: now also J16.8 (Pin_8)
- net R renamed R_1
- net RN renamed RN_1
- net SIG+ renamed SIG_1+
- net SIG_1+: now also J16.6 (Pin_6)
- net SIG- renamed SIG_1-
- net SIG_1-: now also J16.7 (Pin_7)
- net T renamed T_1
- net TN renamed TN_1
- new net: D10.2 (A), D11.1 (K), D9.1 (K), Q4.1 (C), R46.1, R52.1, U9.2 (-)
- new net: C16.2, C19.1, C21.1, Q4.2 (B), R41.1
- new net: C23.1, C24.1, Q4.3 (E), R51.2, R57.1
- new net: RV2.2, U10.1, U10.5 (+)
- new net: R53.2, R55.2, U10.2 (-)
- new net: R54.2, R56.1, U10.3 (+)
- new net: R48.2, R50.2, SW4.7 (A)
- new net: D7.2 (A), R32.2
- new net: C25.2, R58.2, R59.1, U9.6 (-)
- new net: C24.2, C27.1, R57.2, R59.2, U9.1
- new net: R54.1, SW4.8 (B)
- new net: SW4.4 (A), U8.5 (+)
- new net: R35.1, SW4.1 (A), SW4.6 (C)
- new net: D10.1 (K), D8.1 (K), D9.2 (A), Q3.1 (C), R43.1, R46.2, U9.3 (+)
- new net: R47.1, U8.1, U8.2 (-)
- new net: R47.2, R49.1, R53.1
- new net: R33.1, R34.1, SW3.2 (B)
- new net: C16.1, J15.2, R33.2, R36.1
- new net: R60.1, RV2.1
- new net: C17.2, C19.2, C20.1, Q3.2 (B), R40.1
- new net: R55.1, U10.6 (-), U10.7
- new net: C25.1, C26.1, R45.2, R58.1, U9.7
- new net: C22.2, SW4.9 (C)
- new net: R32.1, SW3.5 (B)
- new net: Q3.3 (E), R42.2, R44.1, R45.1
- new net: C15.1, R35.2
- new net: C17.1, J15.3, R34.2, R36.2
- new net: R48.1, U8.6 (-), U8.7
- new net: C26.2, SW4.10 (A)
- new net: R44.2, RV2.1
- new net: C23.2, RV2.2, RV2.3
- new net MON_2: D12.1 (K), J16.11 (Pin_11)
- new net RN_2: J15.RN, SW4.11 (B)
- new net R_2: J15.R, SW4.3 (C), U8.3 (+)
- new net SIG_2+: D12.2 (A), J16.9 (Pin_9), R61.1, RV2.3
- new net TN_2: C27.2, J15.TN
- new net T_2: J15.T, SW4.5 (B)
Other:
- note added: "(simulated approx. gain) stage 1 gain: +5dB to +35dB stage 2 gain: -4dB to +36dB stage 2 unbalanced gain: -4dB to +36dB mic/line pad: -6dB inst gain: 4dB mic gain: -5dB to +65db line gain: -10db to +30db inst gain: +0db to +40db"
- note added: "inst and line input 1"
- note added: "inst and line input 2"
- note added: "instrument input gain (+4dB) and filter ref: 1. pg 354, fig. 12.5"
- note added: "mic input 2"
- note added: "phantom power indicator 1"
- note added: "phantom power indicator 2"
- note added: "phantom power switch 1"
- note added: "phantom power switch 2"
- note added: "unbalanced input converts to balanced, +6dB -10dB to +30dB per phase = -4dB to +36dB"
- note removed: "(simulated approx. gain) stage 1 gain: +5dB to +35dB stage 2 gain: -4dB to +36dB stage 2 unbalanced gain: -10dB to +30dB mic/line pad: -6dB inst gain: 10dB mic gain: -5dB to +65db line gain: -10db to +30db inst gain: +0db to +40db"
- note removed: "inst and line input"
- note removed: "instrument input gain (+10dB) and filter ref: 1. pg 354, fig. 12.5"
- note removed: "phantom power indicator"
- note removed: "phantom power switch"
- note removed: "use with another input"
- moved on the sheet: C1, C10, C11, C12, C13, C14, C2, C3, C4, C5, C6, C7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

Commit message: phantom switch (#6)
Parts:
- removed D1, D7: LED, symbol Device:LED
- removed R1, R32: 330, symbol Device:R_US
- removed SW1, SW3: SW_DPDT_x2, symbol Switch:SW_DPDT_x2
Connections:
- net +48V is gone; now on net phantom: J16.1 (Pin_1)
- net phantom: now reaches R33.1, R34.1
- net phantom: now also R2.1, R4.1
Other:
- note removed: "phantom power indicator 1"
- note removed: "phantom power indicator 2"
- note removed: "phantom power switch 1"
- note removed: "phantom power switch 2"
