File: kicad/om_phonesout/om_phonesout.kicad_sch (KiCad schematic)
At the start: 38 parts, among them J1 AudioJack3, U1 Opamp_Quad, U2 Opamp_Quad

Commit message: headphone driver (#7)
Parts:
- removed C1, C8: 470uF, symbol Device:C_Polarized_US
- removed C10, C11, C3, C4: 100pF, symbol Device:C
- removed C2, C9: 10uF, symbol Device:C_Polarized_US
- removed C3 (x2): 100uF, symbol Device:C
- removed C5 (x2): 220uF, symbol Device:C_Polarized_US
- removed J1: AudioJack3, symbol Connector_Audio:AudioJack3
- removed R1, R16: 47k, symbol Device:R_US
- removed R17, R19, R2, R20, R21, R22, R4, R5, R6, R7: 1k, symbol Device:R_US
- removed R18, R3: 2k2, symbol Device:R_US
- removed R23, R24, R8, R9: 10, symbol Device:R_US
- removed R8 (x2): 100, symbol Device:R_US
- removed R8 (x2): 22k, symbol Device:R_US
- removed RV1: 2k, symbol openmic:R_Potentiometer_US_Dual
- removed U1, U2: Opamp_Quad, symbol Device:Opamp_Quad
- added C43, C44: C_Polarized_US, symbol Device:C_Polarized_US
- added C45, C46: 10uF, symbol Device:C_Polarized_US
- added C47, C48: 100pF, symbol Device:C
- added C49, C50: 47uF, symbol Device:C_Polarized_US
- added J23: Conn_01x05_Pin, symbol Connector:Conn_01x05_Pin
- added J24: AudioJack3, symbol Connector_Audio:AudioJack3
- added R84, R85: 47k, symbol Device:R_US
- added R86, R87, R88, R89: 1k, symbol Device:R_US
- added R90, R92: 1k5, symbol Device:R_US
- added R91, R93: 4k7, symbol Device:R_US
- added RV4: 2k, symbol openmic:R_Potentiometer_US_Dual
- added U14, U15: NE5532, symbol Amplifier_Operational:NE5532
- added U16: OPA1688, symbol openmic:OPA1688
Connections:
- net Earth: now also J23.3 (Pin_3), J24.S, R84.1, R85.1, U14.5 (+), U15.5 (+), U16.3 (+), U16.6 (-)
- new net: C48.2, C50.1, R89.2, RV4.3, U15.7
- new net: C50.2, R92.1
- new net: C47.2, C49.1, R88.2, RV4.3, U14.7
- new net: C49.2, R90.1
- new net: C46.2, R85.2, U15.3 (+)
- new net: R87.1, U15.1, U15.2 (-)
- new net: R90.2, R91.1, U16.2 (-)
- new net: J24.T, R91.2, U16.1
- new net: C46.1, RV4.2
- new net: R86.1, U14.1, U14.2 (-)
- new net: C47.1, R86.2, R88.1, U14.6 (-)
- new net: C48.1, R87.2, R89.1, U15.6 (-)
- new net: J24.R, R93.2, U16.7
- new net: C43.2, RV4.1
- new net: C45.2, R84.2, U14.3 (+)
- new net: R92.2, R93.1, U16.5 (+)
- new net: C44.2, RV4.1
- new net: C45.1, RV4.2
- new net +15V: J23.1 (Pin_1), U14.8 (V+), U15.8 (V+), U16.8 (V+)
- new net -15V: J23.2 (Pin_2), U14.4 (V-), U15.4 (V-), U16.4 (V-)
- new net IN_L: C43.1, J23.4 (Pin_4)
- new net IN_R: C44.1, J23.5 (Pin_5)
Other:
- note added: "Baxandall amp Gain: -inf to 0dB"
- note added: "Headphone driver Gain: +10dB"
- note removed: "Baxandall amp"
- note removed: "optional: add another quad op amp for additional drive"
