File: kicad-test/power/power/power.kicad_sch (KiCad schematic)
At the start: 95 parts, among them J1 EN_3V3, J10 GND, J11 Conn_01x04_Pin, J12 GND2, J13 USB_C_Receptacle_USB2.0_16P, J14 USB_C_Receptacle_USB2.0_16P, J2 EN_1V8_0V9, J3 EN_PH, J4 EN_15V, J5 EN_0V9, J6 +15V, J7 -15V, J8 +5V, J9 +48V, T1 475uH, U1 TPS62172DSG, U10 TPS2116DRL, U2 TPS62171DSG, U3 SN6505BDBV, U4 TPS61391, U5 TPS7A2009, U6 TPS7A39, U7 TPS7A4101, U8 CH224K, U9 PTN5150AHXMP

Commit message: power board layout updates
Parts:
- C20, C21: footprint Capacitor_SMD:C_0805_2012Metric_Pad1.18x1.45mm_HandSolder -> Capacitor_SMD:C_1210_3225Metric_Pad1.33x2.70mm_HandSolder
Changed lines of the file:
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@@
 			)
 		)
-		(property "Footprint" "Capacitor_SMD:C_0805_2012Metric_Pad1.18x1.45mm_HandSolder"
+		(property "Footprint" "Capacitor_SMD:C_1210_3225Metric_Pad1.33x2.70mm_HandSolder"
 			(at 221.9452 205.74 0)
 			(hide yes)
@@
 			)
 		)
-		(property "Footprint" "Capacitor_SMD:C_0805_2012Metric_Pad1.18x1.45mm_HandSolder"
+		(property "Footprint" "Capacitor_SMD:C_1210_3225Metric_Pad1.33x2.70mm_HandSolder"
 			(at 233.3752 205.74 0)
 			(hide yes)
