File: kicad-test/input/input.kicad_sch (KiCad schematic)
At the start: 107 parts, among them J1 Conn_01x02_Pin, J2 Conn_01x06_Pin, J3 NCJ10FI-H-0, J4 Conn_01x02_Pin, J5 Conn_01x02_Pin, Q5 CSD13380F3, SW1 INST_SW, SW10 GAIN_2, SW11 GAIN_3, SW2 TRS_SW, SW7 GAIN_0, SW8 SW_DPST_x2, SW9 GAIN_1, U1 THAT5263, U14 INA1650, U2 THAT1580, U3 OPA1637, U5 OPA1612AxD, U6 OPA1642

Commit message: add footprints
Parts:
- removed C24, C30: 100pF, Capacitor_SMD:C_0603_1608Metric_Pad1.08x0.95mm_HandSolder, symbol Device:C
- removed D14, D15: BAV99, Package_TO_SOT_SMD:SOT-23, symbol Diode:BAV99
- removed R11, R14: 1k2, Resistor_SMD:R_0603_1608Metric_Pad0.98x0.95mm_HandSolder, symbol Device:R_US
- added C27, C32: 100pF, Capacitor_SMD:C_0603_1608Metric_Pad1.08x0.95mm_HandSolder, symbol Device:C
- added D11, D12: VTVS19ASMF, symbol Device:D_TVS
- added J6: OUT_BIAS, symbol Connector:Conn_01x02_Pin
- added J7: AUDIO_OUT, symbol Connector:Conn_01x02_Pin
- added JP3, JP4: SolderJumper_2_Open, symbol Jumper:SolderJumper_2_Open
- added R125, R126: 5k, Resistor_SMD:R_0603_1608Metric_Pad0.98x0.95mm_HandSolder, symbol Device:R_US
- added R15, R38: 1k2, Resistor_SMD:R_0603_1608Metric_Pad0.98x0.95mm_HandSolder, symbol Device:R_US
- J1: value Conn_01x02_Pin -> 5263_GPO
- J2: value Conn_01x06_Pin -> 5263
- J4: value Conn_01x02_Pin -> XLR_SIG
- J5: value Conn_01x02_Pin -> TRS_SIG
Connections:
- net GNDA: now also C27.2, C32.1, D11.1 (A1), D12.2 (A2), JP3.1 (A), JP4.1 (A), R15.2, R38.1
- net at C26.1, R10.2, U2.7 (IN1): now also C27.1, D11.2 (A2), R15.1
- net at C26.2, R13.2, U2.10 (IN2): now also C32.2, D12.1 (A1), R38.2
- net OUT_1_N: no longer names the net of C50.1
- net OUT_1_N: now also J7.2 (Pin_2), R126.2
- net OUT_1_P: no longer names the net of C51.1
- net OUT_1_P: now also J7.1 (Pin_1), R125.2
- new net: J6.2 (Pin_2), JP3.2 (B), R126.1
- new net: J6.1 (Pin_1), JP4.2 (B), R125.1
Other:
- note added: "1100 = -12dB 0100 = -6dB 0000 = 0dB 0010 = +6dB 0011 = +12dB"

Commit message: add footprints
Parts:
- D1, D10, D2, D3, D4, D5, D6, D7, D8, D9: footprint (none) -> LED_SMD:LED_0805_2012Metric_Pad1.15x1.40mm_HandSolder
- J1, J4, J5, J6, J7: footprint (none) -> Connector_PinHeader_2.54mm:PinHeader_1x02_P2.54mm_Vertical
- J2: footprint (none) -> Connector_PinHeader_2.54mm:PinHeader_1x06_P2.54mm_Vertical
- JP1, JP2, JP3, JP4, JP5, JP6: footprint (none) -> Jumper:SolderJumper-2_P1.3mm_Open_RoundedPad1.0x1.5mm
Other:
- moved on the sheet: D1, D2, D3, R22, R27, R30, SW1D, SW2C, SW2D

Commit message: added mcu test schematic
Parts:
- removed J4: XLR_SIG, Connector_PinHeader_2.54mm:PinHeader_1x02_P2.54mm_Vertical, symbol Connector:Conn_01x02_Pin
- removed J5: TRS_SIG, Connector_PinHeader_2.54mm:PinHeader_1x02_P2.54mm_Vertical, symbol Connector:Conn_01x02_Pin
- added J8: XLR_SIG, Connector_PinHeader_2.54mm:PinHeader_1x03_P2.54mm_Vertical, symbol Connector:Conn_01x03_Pin
- added J9: TRS_SIG, Connector_PinHeader_2.54mm:PinHeader_1x03_P2.54mm_Vertical, symbol Connector:Conn_01x03_Pin
Connections:
- net GNDA: now also J8.3 (Pin_3), J9.3 (Pin_3)
- net at C37.1, JP6.2 (B), SW1.5 (B): now also J9.1 (Pin_1)
- net at C25.2, C28.1, C29.1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: now also J8.2 (Pin_2)
- net at C36.1, D65.3 (K), JP5.2 (B)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: now also J9.2 (Pin_2)
- net at C22.1, C23.1, C25.1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: now also J8.1 (Pin_1)

Commit message: sch updates
Parts:
- added J4: 48V_PH, symbol Connector:Conn_01x02_Pin
- added JP7, JP8: SolderJumper_2_Bridged, symbol Jumper:SolderJumper_2_Bridged
Connections:
- net at C51.1, J7.1 (Pin_1): now also JP7.2 (B); no longer R125.2
- net at C50.1, J7.2 (Pin_2): now also JP8.2 (B); no longer R126.2
- net +48V_PH: no longer names the net of R8.2, R9.1
- net +48V_PH: now also J4.1 (Pin_1), J4.2 (Pin_2)
- new net: JP8.1 (A), R126.2
- new net: JP7.1 (A), R125.2
Other:
- moved on the sheet: J6, JP3, JP4, R125, R126

Commit message: footprint assignments
Parts:
- removed R31: 47k, Resistor_SMD:R_0603_1608Metric_Pad0.98x0.95mm_HandSolder, symbol Device:R_US
- removed SW10: GAIN_2, symbol Switch:SW_DPST_x2
- removed SW11: GAIN_3, symbol Switch:SW_DPST_x2
- removed SW7: GAIN_0, symbol Switch:SW_DPST_x2
- removed SW8: SW_DPST_x2, symbol Switch:SW_DPST_x2
- removed SW9: GAIN_1, symbol Switch:SW_DPST_x2
- removed U1: THAT5263, Package_DFN_QFN:QFN-24-1EP_5x5mm_P0.65mm_EP3.4x3.4mm, symbol Audio:THAT5263
- removed U6: OPA1642, Package_SO:VSSOP-8_3x3mm_P0.65mm, symbol Device:Opamp_Dual
- added J5: Conn_01x04_Pin, symbol Connector:Conn_01x04_Pin
- added SW12: IN_EN, openmic:DPDT_SW, symbol openmic:SW_DPDT_x2
- added SW3: GAIN_0, openmic:DPDT_SW, symbol openmic:SW_DPDT_x2
- added SW4: GAIN_1, openmic:DPDT_SW, symbol openmic:SW_DPDT_x2
- added SW5: GAIN_2, openmic:DPDT_SW, symbol openmic:SW_DPDT_x2
- added SW6: GAIN_3, openmic:DPDT_SW, symbol openmic:SW_DPDT_x2
- added TP1: INST_TP, TestPoint:TestPoint_Pad_D2.5mm, symbol Connector:TestPoint_Alt
- added TP2: LINE_TP, TestPoint:TestPoint_Pad_D2.5mm, symbol Connector:TestPoint_Alt
- added TP3: LINE_INST_N_TP, TestPoint:TestPoint_Pad_D2.5mm, symbol Connector:TestPoint_Alt
- added TP4: LINE_INST_P_TP, TestPoint:TestPoint_Pad_D2.5mm, symbol Connector:TestPoint_Alt
- added TP5: MIC_P_TP, TestPoint:TestPoint_Pad_D2.5mm, symbol Connector:TestPoint_Alt
- added TP6: MIC_N_TP, TestPoint:TestPoint_Pad_D2.5mm, symbol Connector:TestPoint_Alt
- added TP7: OUT_N_TP, TestPoint:TestPoint_Pad_D2.5mm, symbol Connector:TestPoint_Alt
- added TP8: OUT_P_TP, TestPoint:TestPoint_Pad_D2.5mm, symbol Connector:TestPoint_Alt
- added U4: OPA1641, Package_SO:SOIC-8_3.9x4.9mm_P1.27mm, symbol Amplifier_Operational:OPA1641
- added U6: THAT5263, Package_DFN_QFN:QFN-24-1EP_5x5mm_P0.65mm_EP3.4x3.4mm, symbol Audio:THAT5263
- C1, C100, C104, C181, C182, C183, C184, C185, C186, C19, C20, C21, C23, C25, C26, C27, C29, C31, C32, C36, C37, C56, C57, C70, C72, C87, C98, C99: footprint Capacitor_SMD:C_0603_1608Metric_Pad1.08x0.95mm_HandSolder -> Capacitor_SMD:C_0805_2012Metric_Pad1.18x1.45mm_HandSolder
- C15: footprint Capacitor_SMD:CP_Elec_8x10.5 -> Capacitor_SMD:CP_Elec_8x10
- C22, C28: footprint Capacitor_SMD:CP_Elec_6.3x5.4 -> Capacitor_SMD:CP_Elec_6.3x5.8
- C50, C51: footprint Capacitor_SMD:CP_Elec_6.3x5.4 -> Capacitor_SMD:CP_Elec_5x5.4
- D11, D12: footprint (none) -> Diode_SMD:D_SMF
- D65, D66: footprint Package_TO_SOT_SMD:SOT-23 -> Package_TO_SOT_SMD:TSOT-23_HandSoldering
- J4: footprint (none) -> Connector_PinHeader_2.54mm:PinHeader_1x02_P2.54mm_Vertical
- JP7, JP8: footprint (none) -> Jumper:SolderJumper-2_P1.3mm_Bridged2Bar_RoundedPad1.0x1.5mm
- R10, R12, R121, R123, R124, R125, R126, R127, R128, R13, R15, R16, R17, R18, R19, R20, R21, R22, R23, R24, R25, R26, R27, R28, R29, R30, R32, R33, R34, R35, R36, R37, R38, R5, R8, R80, R87, R9: footprint Resistor_SMD:R_0603_1608Metric_Pad0.98x0.95mm_HandSolder -> Resistor_SMD:R_0805_2012Metric_Pad1.20x1.40mm_HandSolder
- SW1, SW2: footprint (none) -> openmic:4PDT_SW
Connections:
- net GNDA is gone; now on net Earth: C181.2, C182.2, C183.2, C184.2, C185.2, C186.2, C20.2, C27.2, C31.2, C32.1, C56.2, C57.2, C72.1, C87.2, C98.1, C99.1, D11.1 (A1), D12.2 (A2), D4.1 (K), D5.1 (K), J3.1, J3.G, J3.RN, J3.S, J3.TN, J8.3 (Pin_3), J9.3 (Pin_3), JP3.1 (A), JP4.1 (A), Q5.2 (S), R12.1, R15.2, R38.1, R80.2, R87.2, SW1.6 (C), U14.12 (REF), U3.2 (VOCM), U5.3 (+), U5.6 (-)
- net GNDD is gone; now on net Earth: C1.2, C19.2, C70.2, D1.1 (K), D10.1 (K), D2.1 (K), D3.1 (K), D6.1 (K), D7.1 (K), D8.1 (K), D9.1 (K), SW1.10 (A), SW2.10 (A)
- net +15V: now also J5.2 (Pin_2), U4.7 (V+), U6.4 (V+)
- net +3V3: now also SW2.12 (C), J5.1 (Pin_1), SW12.3 (C), SW12.6 (C), U6.15 (VDD); no longer SW1.12 (C)
- net -15V: now also J5.3 (Pin_3), U4.4 (V-), U6.25 (PAD), U6.3 (V-)
- net Earth: now also J5.4 (Pin_4), SW12.1 (A), SW12.4 (A), SW3.4 (A), SW4.4 (A), SW5.4 (A), SW6.4 (A), U6.16 (DGND)
- net at R124.1, R29.1, U3.4 (VOUT+): now also TP8.1
- net at SW1.7 (A), U14.13 (OUT): now also TP2.1
- net at R24.1, SW1.8 (B): now also SW3.2 (B)
- net at SW1.9 (C): now also TP1.1, U4.2 (-), U4.6
- net at R121.2: now also U4.3 (+)
- net at R19.2, R20.1: now also SW5.2 (B)
- net at R20.2, R21.1: now also SW5.3 (C), SW6.2 (B)
- net at J2.3 (Pin_3): now also U6.11 (~{CS})
- net at J2.4 (Pin_4): now also U6.12 (SCLK)
- net at J2.5 (Pin_5): now also U6.13 (DIN)
- net at J2.6 (Pin_6): now also U6.14 (DOUT)
- net at J2.1 (Pin_1): now also U6.17 (BSY_CH1)
- net at J2.2 (Pin_2): now also U6.18 (BSY_CH2)
- net at J1.1 (Pin_1): now also U6.19 (GPO_CH1)
- net at J1.2 (Pin_2): now also U6.20 (GPO_CH2)
- net at R24.2, R25.1: now also SW3.3 (C), SW4.2 (B)
- net at R36.2: now also SW5.5 (B)
- net at SW1.11 (B): now also R22.1; no longer SW2.12 (C)
- net at R127.2, SW2.3 (C), U5.7: now also TP4.1
- net at R35.2: now also SW4.5 (B)
- net at R5.1, U2.15 (Rg2): now also U6.8 (RG2_CH1), U6.9 (RB_CH1)
- net at C15.2, R5.2: now also U6.7 (RG1_CH1)
- net TRS_EN: now reaches SW2.11 (B)
- net TRS_EN: now also SW1.12 (C), SW3.6 (C), SW4.6 (C), SW5.6 (C), SW6.6 (C); no longer R22.1
- net at R128.1, R21.2, SW2.6 (C)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: now also SW6.3 (C), TP3.1
- net at R25.2, R26.1: now also SW4.3 (C)
- net at C15.1, U2.6 (Rg1): now also U6.6 (RA_CH1)
- net at R37.2: now also SW6.5 (B)
- net at Q5.1 (G): now also SW12.2 (B)
- net at R33.1: now also SW12.5 (B)
- net at R123.1, R17.2, U3.5 (VOUT-): now also TP7.1
- net at R34.2: now also SW3.5 (B)
- net MIC_1_N renamed MIC_N
- net MIC_N: now also TP6.1, U6.10 (IN2_CH1)
- net MIC_1_P renamed MIC_P
- net MIC_P: now also TP5.1, U6.5 (IN1_CH1)
Other:
- moved on the sheet: D1, D10, D6, D7, D8, D9, R22, R33, R34, R35, R36, R37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

Commit message: pcb layout
Parts:
- removed JP3, JP4: SolderJumper_2_Open, Jumper:SolderJumper-2_P1.3mm_Open_RoundedPad1.0x1.5mm, symbol Jumper:SolderJumper_2_Open
- removed Q5: CSD13380F3, Package_DFN_QFN:Texas_PicoStar_DFN-3_0.69x0.60mm, symbol Transistor_FET:CSD13380F3
- added Q2: BSS138, Package_TO_SOT_SMD:SOT-23, symbol Transistor_FET:BSS138
- J1: renamed from J5; footprint (none) -> Connector_PinHeader_2.54mm:PinHeader_1x04_P2.54mm_Vertical
- TP1: renamed from TP2; footprint TestPoint:TestPoint_Pad_D2.5mm -> TestPoint:TestPoint_Pad_D1.0mm
- TP2: renamed from TP1; footprint TestPoint:TestPoint_Pad_D2.5mm -> TestPoint:TestPoint_Pad_D1.0mm
- TP3: renamed from TP5; footprint TestPoint:TestPoint_Pad_D2.5mm -> TestPoint:TestPoint_Pad_D1.0mm
- TP4: renamed from TP6; footprint TestPoint:TestPoint_Pad_D2.5mm -> TestPoint:TestPoint_Pad_D1.0mm
- TP5: renamed from TP4; footprint TestPoint:TestPoint_Pad_D2.5mm -> TestPoint:TestPoint_Pad_D1.0mm
- TP6: renamed from TP3; footprint TestPoint:TestPoint_Pad_D2.5mm -> TestPoint:TestPoint_Pad_D1.0mm
- TP7, TP8: footprint TestPoint:TestPoint_Pad_D2.5mm -> TestPoint:TestPoint_Pad_D1.0mm
- renumbered C57 to C1, C27 to C10, C32 to C11, C100 to C12, C104 to C13, C26 to C14, C181 to C15, C182 to C16, C15 to C17, C98 to C18, C72 to C19, C36 to C2, C87 to C20, C99 to C21, C19 to C22, C1 to C23, C20 to C24, C31 to C25, C21 to C26, C183 to C27, C184 to C28, C70 to C29, C37 to C3, C185 to C30, C186 to C31, C50 to C32, C51 to C33, C23 to C4, C29 to C5, C56 to C6, C25 to C7, C22 to C8, C28 to C9, D4 to D1, D8 to D10, D7 to D11, D2 to D12, D3 to D13, D6 to D14, D5 to D2, D1 to D3, D65 to D4, D66 to D5, D11 to D6, D12 to D7, D10 to D8, J3 to J2, J9 to J3, J8 to J4, J4 to J5, J2 to J6, J1 to J7, J6 to J8, J7 to J9, JP6 to JP1, JP5 to JP2, JP1 to JP3, JP2 to JP4, JP7 to JP5, JP8 to JP7, R32 to R1, R38 to R10, R121 to R11, R87 to R12, R12 to R13, R5 to R14, R24 to R15, R25 to R16, R26 to R17, R19 to R18, R20 to R19, R18 to R2, R21 to R20, R37 to R21, R36 to R22, R35 to R23, R34 to R24, R128 to R25, R127 to R26, R30 to R28, R33 to R29, R8 to R3, R23 to R30, R16 to R31, R28 to R32, R29 to R33, R17 to R34, R123 to R35, R124 to R36, R125 to R37, R126 to R38, R22 to R4, R9 to R5, R10 to R6, R13 to R7, R80 to R8, R15 to R9, SW2 to SW1, SW1 to SW2, SW12 to SW7, U14 to U1, U4 to U2, U6 to U3, U2 to U4, U3 to U6
Connections:
- net Earth: now also J8.2 (Pin_2), Q2.2 (S)
- net at R38.1: now also J8.1 (Pin_1), R37.1; no longer J8.2 (Pin_2)
- net at C12.1: now also U1.4 (IN-); no longer U1.2 (IN+)
- net at C13.1: now also U1.2 (IN+); no longer U1.4 (IN-)
- net at SW7.2 (B): now also Q2.1 (G)
- net at U6.7 (PD_N): now also Q2.3 (D)
Other:
- moved on the sheet: D2, J8
