File: kicad-test/input/input.kicad_pcb (KiCad board)
At the start: 2 copper layers, 123 parts, among them J1 5263_GPO, J2 5263, J3 NCJ10FI-H-0, J4 48V_PH, J6 OUT_BIAS, J7 AUDIO_OUT, J8 XLR_SIG, J9 TRS_SIG, Q5 CSD13380F3, SW1 INST_SW, SW12 IN_EN, SW2 TRS_SW, SW3 GAIN_0, SW4 GAIN_1, SW5 GAIN_2, SW6 GAIN_3, U14 INA1650, U2 THAT1580, U3 OPA1637, U4 OPA1641, U5 OPA1612AxD, U6 THAT5263

Commit message: pcb layout
Parts:
- removed the JP3 at (73.0, 78.6)
- removed the JP4 at (73.0, 82.1)
- removed JP8: SolderJumper_2_Bridged, Jumper:SolderJumper-2_P1.3mm_Bridged2Bar_RoundedPad1.0x1.5mm
- removed Q5: CSD13380F3, Package_DFN_QFN:Texas_PicoStar_DFN-3_0.69x0.60mm
- added J1: Conn_01x04_Pin, Connector_PinHeader_2.54mm:PinHeader_1x04_P2.54mm_Vertical, F.Cu at (58.4, 110.5)
- added JP5: SolderJumper_2_Bridged, Jumper:SolderJumper-2_P1.3mm_Bridged2Bar_RoundedPad1.0x1.5mm, F.Cu at (127.6, 124.5)
- added Q2: BSS138, Package_TO_SOT_SMD:SOT-23, F.Cu at (127.3, 127.7)
- TP1: renamed from TP2; footprint TestPoint:TestPoint_Pad_D2.5mm -> TestPoint:TestPoint_Pad_D1.0mm
- TP2: renamed from TP1; footprint TestPoint:TestPoint_Pad_D2.5mm -> TestPoint:TestPoint_Pad_D1.0mm
- TP3: renamed from TP5; footprint TestPoint:TestPoint_Pad_D2.5mm -> TestPoint:TestPoint_Pad_D1.0mm
- TP4: renamed from TP6; footprint TestPoint:TestPoint_Pad_D2.5mm -> TestPoint:TestPoint_Pad_D1.0mm
- TP5: renamed from TP4; footprint TestPoint:TestPoint_Pad_D2.5mm -> TestPoint:TestPoint_Pad_D1.0mm
- TP6: renamed from TP3; footprint TestPoint:TestPoint_Pad_D2.5mm -> TestPoint:TestPoint_Pad_D1.0mm
- TP7, TP8: footprint TestPoint:TestPoint_Pad_D2.5mm -> TestPoint:TestPoint_Pad_D1.0mm
- moved R27 133.3 mm to (118.1, 158.8)
- moved D13 133.0 mm to (132.1, 158.8)
- moved D12 132.2 mm to (122.6, 158.8)
- moved D3 129.8 mm to (52.8, 158.8)
- moved R28 129.7 mm to (127.6, 158.8)
- moved R24 127.5 mm to (65.8, 158.8)
- moved D11 125.0 mm to (70.5, 158.8)
- moved R23 124.9 mm to (78.5, 158.8)
- moved R21 123.9 mm to (104.1, 158.8)
- moved R22 123.8 mm to (91.4, 158.8)
- moved R16 122.9 mm to (121.3, 139.7), turned to 90 degrees
- moved R17 121.5 mm to (123.8, 139.7), turned to 90 degrees
- moved D10 121.3 mm to (83.2, 158.8)
- moved D9 119.1 mm to (95.9, 158.8)
- moved D8 118.2 mm to (108.6, 158.8)
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- renumbered C57 to C1, C27 to C10, C32 to C11, C100 to C12, C104 to C13, C26 to C14, C181 to C15, C182 to C16, C15 to C17, C98 to C18, C72 to C19, C36 to C2, C87 to C20, C99 to C21, C19 to C22, C1 to C23, C20 to C24, C31 to C25, C21 to C26, C183 to C27, C184 to C28, C70 to C29, C37 to C3, C185 to C30, C186 to C31, C50 to C32, C51 to C33, C23 to C4, C29 to C5, C56 to C6, C25 to C7, C22 to C8, C28 to C9, D4 to D1, D8 to D10, D7 to D11, D2 to D12, D3 to D13, D6 to D14, D5 to D2, D1 to D3, D65 to D4, D66 to D5, D11 to D6, D12 to D7, D10 to D8, J3 to J2, J9 to J3, J8 to J4, J4 to J5, J2 to J6, J1 to J7, J6 to J8, J7 to J9, JP6 to JP1, JP5 to JP2, JP1 to JP3, JP2 to JP4, R32 to R1, R38 to R10, R121 to R11, R87 to R12, R12 to R13, R5 to R14, R24 to R15, R25 to R16, R26 to R17, R19 to R18, R20 to R19, R18 to R2, R21 to R20, R37 to R21, R36 to R22, R35 to R23, R34 to R24, R128 to R25, R127 to R26, R30 to R28, R33 to R29, R8 to R3, R23 to R30, R16 to R31, R28 to R32, R29 to R33, R17 to R34, R123 to R35, R124 to R36, R125 to R37, R126 to R38, R22 to R4, R9 to R5, R10 to R6, R13 to R7, R80 to R8, R15 to R9, SW2 to SW1, SW1 to SW2, SW12 to SW7, U14 to U1, U4 to U2, U6 to U3, U2 to U4, U3 to U6
Connections:
- C12 pad 1: Net-(U14A-IN+) -> Net-(U1A-IN-)
- C13 pad 1: Net-(U14A-IN-) -> Net-(U1A-IN+)
- C32 pad 1: Net-(J7-Pin_2) (its old number) -> Net-(J9-Pin_2)
- C33 pad 1: Net-(J7-Pin_1) (its old number) -> Net-(J9-Pin_1)
- J8 pad 1: Net-(J6-Pin_1) (its old number) -> Net-(J8-Pin_1)
- J8 pad 2: Net-(J6-Pin_2) (its old number) -> Earth
- J9 pad 1: Net-(J7-Pin_1) (its old number) -> Net-(J9-Pin_1)
- J9 pad 2: Net-(J7-Pin_2) (its old number) -> Net-(J9-Pin_2)
- JP7 pad 2: Net-(J7-Pin_1) (its old number) -> Net-(J9-Pin_2)
- R37 pad 1: Net-(J6-Pin_1) (its old number) -> Net-(J8-Pin_1)
- R37 pad 2: Net-(JP7-A) -> Net-(JP5-A)
- R38 pad 1: Net-(J6-Pin_2) (its old number) -> Net-(J8-Pin_1)
- R38 pad 2: Net-(JP8-A) -> Net-(JP7-A)
- U1 pad 2: Net-(U14A-IN+) -> Net-(U1A-IN+)
- U1 pad 4: Net-(U14A-IN-) -> Net-(U1A-IN-)
Routing:
- net -15V: track 0.00 -> 183.6 mm, vias 0 -> 4
- net +3V3: track 0.00 -> 181.8 mm, vias 0 -> 3
- net +15V: track 0.00 -> 181.6 mm, vias 0 -> 6
- net Earth: track 0.00 -> 118.8 mm, vias 0 -> 42
- net Net-(J3-Pin_2): track 0.00 -> 97.3 mm, vias 0 -> 1
- net Net-(SW2C-B): track 0.00 -> 85.3 mm, vias 0 -> 1
- net /TRS_EN: track 0.00 -> 80.7 mm, vias 0 -> 2
- net Net-(SW3A-C): track 0.00 -> 80.4 mm, vias 0 -> 1
- net Net-(J3-Pin_1): track 0.00 -> 67.8 mm, vias 0 -> 1
- net Net-(SW2C-C): track 0.00 -> 67.4 mm, vias 0 -> 2
- net Net-(SW2C-A): track 0.00 -> 65.8 mm, vias 0 -> 4
- net Net-(SW2A-A): track 0.00 -> 61.0 mm, vias 0 -> 1
- net Net-(SW2A-C): track 0.00 -> 59.3 mm, vias 0 -> 1
- net Net-(SW5A-C): track 0.00 -> 58.8 mm, vias 0 -> 3
- net Net-(SW5A-B): track 0.00 -> 57.1 mm, vias 0 -> 3
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- added copper zone on B.Cu, net Earth
Other:
- board outline added: 100 x 61 mm
- board text added: "+"
- board text added: "+15V"
- board text added: "+3V3"
- board text added: "+48V"
- board text added: "-"
- board text added: "-15V"
- board text added: "BIAS"
- board text added: "BSY1"
- board text added: "BSY2"
- board text added: "CS"
- board text added: "DIN"
- board text added: "DOUT"
- board text added: "G"
- board text added: "G0"
- board text added: "G1"
- board text added: "G2"
- board text added: "G3"
- board text added: "GND"
- board text added: "GPO1"
- board text added: "GPO2"
- board text added: "INST"
- board text added: "OUT"
- board text added: "SCLK"
- board text added: "TRS"
- board text added: "XLR"

Commit message: add aisler sponsorship
Routing:
- net Earth: track 118.8 -> 285.1 mm, vias 42 -> 128
