File: kicad-test/power v2/select.kicad_sch (KiCad schematic)
At the start: 7 parts, among them U3 TPS2116DRL

Commit message: pcb layout
Parts:
- removed TP5: VOUT, TestPoint:TestPoint_Loop_D3.80mm_Drill2.0mm, symbol Connector:TestPoint
- renumbered C22 to C20, C20 to C21, C21 to C22, R9 to R10, R8 to R9
Changed lines of the file:
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@@
 		(dnp no)
 		(fields_autoplaced yes)
-		(property "Reference" "R9"
+		(property "Reference" "R10"
 			(at 105.41 82.5499 0)
 			(show_name no)
@@
 			(project "power v2"
 				(path "/7765ea03-990c-41e2-8b83-b7e84578cc41/563617a4-17e3-447c-9915-8985ac21500e"
-					(reference "R9")
+					(reference "R10")
 					(unit 1)
 				)
@@
 		(dnp no)
 		(fields_autoplaced yes)
-		(property "Reference" "#PWR023"
+		(property "Reference" "#PWR026"
 			(at 102.87 92.71 0)
 			(hide yes)
@@
 			(project "power v2"
 				(path "/7765ea03-990c-41e2-8b83-b7e84578cc41/563617a4-17e3-447c-9915-8985ac21500e"
-					(reference "#PWR023")
+					(reference "#PWR026")
 					(unit 1)
 				)
@@
 		(dnp no)
 		(fields_autoplaced yes)
-		(property "Reference" "#PWR026"
+		(property "Reference" "#PWR030"
 			(at 163.83 85.09 0)
 			(hide yes)
@@
 			(project "power v2"
 				(path "/7765ea03-990c-41e2-8b83-b7e84578cc41/563617a4-17e3-447c-9915-8985ac21500e"
-					(reference "#PWR026")
-					(unit 1)
-				)
-			)
-		)
-	)
-	(symbol
-		(lib_id "Connector:TestPoint")
-		(at 163.83 73.66 0)
-		(unit 1)
-		(body_style 1)
-		(exclude_from_sim no)
-		(in_bom yes)
-		(on_board yes)
-		(in_pos_files yes)
-		(dnp no)
-		(fields_autoplaced yes)
-		(property "Reference" "TP5"
-			(at 166.37 69.0879 0)
-			(show_name no)
-			(do_not_autoplace no)
-			(effects
-				(font
-					(size 1.27 1.27)
-				)
-				(justify left)
-			)
-		)
-		(property "Value" "VOUT"
-			(at 166.37 71.6279 0)
-			(show_name no)
-			(do_not_autoplace no)
-			(effects
-				(font
-					(size 1.27 1.27)
-				)
-				(justify left)
-			)
-		)
-		(property "Footprint" "TestPoint:TestPoint_Loop_D3.80mm_Drill2.0mm"
-			(at 168.91 73.66 0)
-			(hide yes)
-			(show_name no)
-			(do_not_autoplace no)
-			(effects
-				(font
-					(size 1.27 1.27)
-				)
-			)
-		)
-		(property "Datasheet" ""
-			(at 168.91 73.66 0)
-			(hide yes)
-			(show_name no)
-			(do_not_autoplace no)
-			(effects
-				(font
-					(size 1.27 1.27)
-				)
-			)
-		)
-		(property "Description" "test point"
-			(at 163.83 73.66 0)
-			(hide yes)
-			(show_name no)
-			(do_not_autoplace no)
-			(effects
-				(font
-					(size 1.27 1.27)
-				)
-			)
-		)
-		(pin "1"
-		)
-		(instances
-			(project "power v2"
-				(path "/7765ea03-990c-41e2-8b83-b7e84578cc41/563617a4-17e3-447c-9915-8985ac21500e"
-					(reference "TP5")
+					(reference "#PWR030")
 					(unit 1)
 				)
@@
 		(dnp no)
 		(fields_autoplaced yes)
-		(property "Reference" "R8"
+		(property "Reference" "R9"
 			(at 105.41 74.9299 0)
 			(show_name no)
@@
 			(project "power v2"
 				(path "/7765ea03-990c-41e2-8b83-b7e84578cc41/563617a4-17e3-447c-9915-8985ac21500e"
-					(reference "R8")
+					(reference "R9")
 					(unit 1)
 				)
@@
 		(dnp no)
 		(fields_autoplaced yes)
-		(property "Reference" "#PWR024"
+		(property "Reference" "#PWR029"
 			(at 148.59 95.25 0)
 			(hide yes)
@@
 			(project "power v2"
 				(path "/7765ea03-990c-41e2-8b83-b7e84578cc41/563617a4-17e3-447c-9915-8985ac21500e"
-					(reference "#PWR024")
+					(reference "#PWR029")
 					(unit 1)
 				)
@@
 		(in_pos_files yes)
 		(dnp no)
-		(property "Reference" "C21"
+		(property "Reference" "C22"
 			(at 166.37 74.9362 0)
 			(show_name no)
@@
 			(project "power v2"
 				(path "/7765ea03-990c-41e2-8b83-b7e84578cc41/563617a4-17e3-447c-9915-8985ac21500e"
-					(reference "C21")
+					(reference "C22")
 					(unit 1)
 				)
@@
 		(in_pos_files yes)
 		(dnp no)
-		(property "Reference" "C20"
+		(property "Reference" "C21"
 			(at 133.35 87.6362 0)
 			(show_name no)
@@
 			(project "power v2"
 				(path "/7765ea03-990c-41e2-8b83-b7e84578cc41/563617a4-17e3-447c-9915-8985ac21500e"
-					(reference "C20")
+					(reference "C21")
 					(unit 1)
 				)
@@
 		(dnp no)
 		(fields_autoplaced yes)
-		(property "Reference" "#PWR025"
+		(property "Reference" "#PWR028"
 			(at 135.89 97.79 0)
 			(hide yes)
@@
 			(project "power v2"
 				(path "/7765ea03-990c-41e2-8b83-b7e84578cc41/563617a4-17e3-447c-9915-8985ac21500e"
-					(reference "#PWR025")
+					(reference "#PWR028")
 					(unit 1)
 				)
@@
 		(in_pos_files yes)
 		(dnp no)
-		(property "Reference" "C22"
+		(property "Reference" "C20"
 			(at 123.19 74.9362 0)
 			(show_name no)
@@
 			(project "power v2"
 				(path "/7765ea03-990c-41e2-8b83-b7e84578cc41/563617a4-17e3-447c-9915-8985ac21500e"
-					(reference "C22")
-					(unit 1)
-				)
+					(reference "C20")
+					(unit 1)
+				)
