File: kicad-test/power v2/usb.kicad_sch (KiCad schematic)
At the start: 19 parts, among them J2 USB_C_Receptacle_USB2.0_16P, J3 D_PIN, U2 TUSB321

Commit message: add footprints
Parts:
- C13, C14, C15, C16, C17, C18, C19: footprint (none) -> Capacitor_SMD:C_0805_2012Metric_Pad1.18x1.45mm_HandSolder
- D1, D2: footprint (none) -> LED_SMD:LED_0805_2012Metric_Pad1.15x1.40mm_HandSolder
- J2: footprint (none) -> Connector_USB:USB_C_Receptacle_HRO_TYPE-C-31-M-12
- J3: footprint (none) -> Connector_PinHeader_2.54mm:PinHeader_1x02_P2.54mm_Vertical
- R1, R2, R6, R7: footprint (none) -> Resistor_SMD:R_0805_2012Metric_Pad1.20x1.40mm_HandSolder
- TP1, TP2, TP3: footprint (none) -> TestPoint:TestPoint_Loop_D3.80mm_Drill2.0mm
Changed lines of the file:
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@@
 			)
 		)
-		(property "Footprint" ""
+		(property "Footprint" "Capacitor_SMD:C_0805_2012Metric_Pad1.18x1.45mm_HandSolder"
 			(at 96.52 96.52 0)
 			(hide yes)
@@
 			)
 		)
-		(property "Footprint" ""
+		(property "Footprint" "LED_SMD:LED_0805_2012Metric_Pad1.15x1.40mm_HandSolder"
 			(at 125.73 49.53 90)
 			(hide yes)
@@
 			)
 		)
-		(property "Footprint" ""
+		(property "Footprint" "TestPoint:TestPoint_Loop_D3.80mm_Drill2.0mm"
 			(at 82.55 41.91 0)
 			(hide yes)
@@
 			)
 		)
-		(property "Footprint" ""
+		(property "Footprint" "Resistor_SMD:R_0805_2012Metric_Pad1.20x1.40mm_HandSolder"
 			(at 125.73 38.1 0)
 			(hide yes)
@@
 			)
 		)
-		(property "Footprint" ""
+		(property "Footprint" "Capacitor_SMD:C_0805_2012Metric_Pad1.18x1.45mm_HandSolder"
 			(at 110.49 96.52 0)
 			(hide yes)
@@
 			)
 		)
-		(property "Footprint" ""
+		(property "Footprint" "Connector_PinHeader_2.54mm:PinHeader_1x02_P2.54mm_Vertical"
 			(at 73.66 57.15 0)
 			(hide yes)
@@
 			)
 		)
-		(property "Footprint" ""
+		(property "Footprint" "Capacitor_SMD:C_0805_2012Metric_Pad1.18x1.45mm_HandSolder"
 			(at 40.64 96.52 0)
 			(hide yes)
@@
 			)
 		)
-		(property "Footprint" ""
+		(property "Footprint" "Resistor_SMD:R_0805_2012Metric_Pad1.20x1.40mm_HandSolder"
 			(at 90.17 58.42 0)
 			(hide yes)
@@
 			)
 		)
-		(property "Footprint" ""
+		(property "Footprint" "Capacitor_SMD:C_0805_2012Metric_Pad1.18x1.45mm_HandSolder"
 			(at 60.96 96.52 0)
 			(hide yes)
@@
 			)
 		)
-		(property "Footprint" ""
+		(property "Footprint" "Capacitor_SMD:C_0805_2012Metric_Pad1.18x1.45mm_HandSolder"
 			(at 71.12 96.52 0)
 			(hide yes)
@@
 			)
 		)
-		(property "Footprint" ""
+		(property "Footprint" "TestPoint:TestPoint_Loop_D3.80mm_Drill2.0mm"
 			(at 125.73 46.99 0)
 			(hide yes)
@@
 			)
 		)
-		(property "Footprint" ""
+		(property "Footprint" "TestPoint:TestPoint_Loop_D3.80mm_Drill2.0mm"
 			(at 138.43 49.53 0)
 			(hide yes)
@@
 			)
 		)
-		(property "Footprint" ""
+		(property "Footprint" "Resistor_SMD:R_0805_2012Metric_Pad1.20x1.40mm_HandSolder"
 			(at 138.43 38.1 0)
 			(hide yes)
@@
 			)
 		)
-		(property "Footprint" ""
+		(property "Footprint" "Connector_USB:USB_C_Receptacle_HRO_TYPE-C-31-M-12"
 			(at 54.61 57.15 0)
 			(hide yes)
@@
 			)
 		)
-		(property "Footprint" ""
+		(property "Footprint" "Capacitor_SMD:C_0805_2012Metric_Pad1.18x1.45mm_HandSolder"
 			(at 50.8 96.52 0)
 			(hide yes)
@@
 			)
 		)
-		(property "Footprint" ""
+		(property "Footprint" "Resistor_SMD:R_0805_2012Metric_Pad1.20x1.40mm_HandSolder"
 			(at 87.63 41.91 0)
 			(hide yes)
@@
 			)
 		)
-		(property "Footprint" ""
+		(property "Footprint" "LED_SMD:LED_0805_2012Metric_Pad1.15x1.40mm_HandSolder"
 			(at 138.43 49.53 90)
 			(hide yes)
@@
 			)
 		)
-		(property "Footprint" ""
+		(property "Footprint" "Capacitor_SMD:C_0805_2012Metric_Pad1.18x1.45mm_HandSolder"
 			(at 81.28 96.52 0)
 			(hide yes)

Commit message: pcb layout
Parts:
- J5: renamed from J3; footprint Connector_PinHeader_2.54mm:PinHeader_1x02_P2.54mm_Vertical -> Connector_PinHeader_1.00mm:PinHeader_1x02_P1.00mm_Vertical
- TP2: renamed from TP3; footprint TestPoint:TestPoint_Loop_D3.80mm_Drill2.0mm -> TestPoint:TestPoint_Pad_1.5x1.5mm
- TP3: renamed from TP1; footprint TestPoint:TestPoint_Loop_D3.80mm_Drill2.0mm -> TestPoint:TestPoint_Pad_1.5x1.5mm
- TP4: renamed from TP2; footprint TestPoint:TestPoint_Loop_D3.80mm_Drill2.0mm -> TestPoint:TestPoint_Pad_1.5x1.5mm
- renumbered D2 to D3, D1 to D4, J2 to J4, R1 to R5, R7 to R6, R2 to R7, R6 to R8
Changed lines of the file:
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@@
 		(dnp no)
 		(fields_autoplaced yes)
-		(property "Reference" "D2"
+		(property "Reference" "D3"
 			(at 128.27 48.1964 90)
 			(show_name no)
@@
 			(project "power v2"
 				(path "/7765ea03-990c-41e2-8b83-b7e84578cc41/8a309907-db9d-4e2b-b4b7-665a29344a77"
-					(reference "D2")
+					(reference "D3")
 					(unit 1)
 				)
@@
 		(in_pos_files yes)
 		(dnp no)
-		(property "Reference" "TP3"
+		(property "Reference" "TP2"
 			(at 75.438 33.782 0)
 			(show_name no)
@@
 			)
 		)
-		(property "Footprint" "TestPoint:TestPoint_Loop_D3.80mm_Drill2.0mm"
+		(property "Footprint" "TestPoint:TestPoint_Pad_1.5x1.5mm"
 			(at 82.55 41.91 0)
 			(hide yes)
@@
 			(project "power v2"
 				(path "/7765ea03-990c-41e2-8b83-b7e84578cc41/8a309907-db9d-4e2b-b4b7-665a29344a77"
-					(reference "TP3")
+					(reference "TP2")
 					(unit 1)
 				)
@@
 		(in_pos_files yes)
 		(dnp no)
-		(property "Reference" "R2"
+		(property "Reference" "R7"
 			(at 127.508 36.068 0)
 			(show_name no)
@@
 			(project "power v2"
 				(path "/7765ea03-990c-41e2-8b83-b7e84578cc41/8a309907-db9d-4e2b-b4b7-665a29344a77"
-					(reference "R2")
+					(reference "R7")
 					(unit 1)
 				)
@@
 		(dnp no)
 		(fields_autoplaced yes)
-		(property "Reference" "J3"
+		(property "Reference" "J5"
 			(at 74.93 57.1499 0)
 			(show_name no)
@@
 			)
 		)
-		(property "Footprint" "Connector_PinHeader_2.54mm:PinHeader_1x02_P2.54mm_Vertical"
+		(property "Footprint" "Connector_PinHeader_1.00mm:PinHeader_1x02_P1.00mm_Vertical"
 			(at 73.66 57.15 0)
 			(hide yes)
@@
 			(project "power v2"
 				(path "/7765ea03-990c-41e2-8b83-b7e84578cc41/8a309907-db9d-4e2b-b4b7-665a29344a77"
-					(reference "J3")
+					(reference "J5")
 					(unit 1)
 				)
@@
 		(in_pos_files yes)
 		(dnp no)
-		(property "Reference" "R7"
+		(property "Reference" "R6"
 			(at 87.63 57.1499 0)
 			(show_name no)
@@
 			(project "power v2"
 				(path "/7765ea03-990c-41e2-8b83-b7e84578cc41/8a309907-db9d-4e2b-b4b7-665a29344a77"
-					(reference "R7")
+					(reference "R6")
 					(unit 1)
 				)
@@
 		(dnp no)
 		(fields_autoplaced yes)
-		(property "Reference" "#PWR014"
+		(property "Reference" "#PWR018"
 			(at 43.18 86.36 0)
 			(hide yes)
@@
 			(project "power v2"
 				(path "/7765ea03-990c-41e2-8b83-b7e84578cc41/8a309907-db9d-4e2b-b4b7-665a29344a77"
-					(reference "#PWR014")
+					(reference "#PWR018")
 					(unit 1)
 				)
@@
 		(in_pos_files yes)
 		(dnp no)
-		(property "Reference" "TP1"
+		(property "Reference" "TP3"
 			(at 131.064 40.64 90)
 			(show_name no)
@@
 			)
 		)
-		(property "Footprint" "TestPoint:TestPoint_Loop_D3.80mm_Drill2.0mm"
+		(property "Footprint" "TestPoint:TestPoint_Pad_1.5x1.5mm"
 			(at 125.73 46.99 0)
 			(hide yes)
@@
 			(project "power v2"
 				(path "/7765ea03-990c-41e2-8b83-b7e84578cc41/8a309907-db9d-4e2b-b4b7-665a29344a77"
-					(reference "TP1")
+					(reference "TP3")
 					(unit 1)
 				)
@@
 		(dnp no)
 		(fields_autoplaced yes)
-		(property "Reference" "#PWR020"
+		(property "Reference" "#PWR024"
 			(at 125.73 58.42 0)
 			(hide yes)
@@
 			(project "power v2"
 				(path "/7765ea03-990c-41e2-8b83-b7e84578cc41/8a309907-db9d-4e2b-b4b7-665a29344a77"
-					(reference "#PWR020")
+					(reference "#PWR024")
 					(unit 1)
 				)
@@
 		(dnp no)
 		(fields_autoplaced yes)
-		(property "Reference" "#PWR021"
+		(property "Reference" "#PWR025"
 			(at 138.43 58.42 0)
 			(hide yes)
@@
 			(project "power v2"
 				(path "/7765ea03-990c-41e2-8b83-b7e84578cc41/8a309907-db9d-4e2b-b4b7-665a29344a77"
-					(reference "#PWR021")
+					(reference "#PWR025")
 					(unit 1)
 				)
@@
 		(dnp no)
 		(fields_autoplaced yes)
-		(property "Reference" "TP2"
+		(property "Reference" "TP4"
 			(at 143.51 43.1799 90)
 			(show_name no)
@@
 			)
 		)
-		(property "Footprint" "TestPoint:TestPoint_Loop_D3.80mm_Drill2.0mm"
+		(property "Footprint" "TestPoint:TestPoint_Pad_1.5x1.5mm"
 			(at 138.43 49.53 0)
 			(hide yes)
@@
 			(project "power v2"
 				(path "/7765ea03-990c-41e2-8b83-b7e84578cc41/8a309907-db9d-4e2b-b4b7-665a29344a77"
-					(reference "TP2")
+					(reference "TP4")
 					(unit 1)
 				)
@@
 		(dnp no)
 		(fields_autoplaced yes)
-		(property "Reference" "R6"
+		(property "Reference" "R8"
 			(at 140.97 36.8299 0)
 			(show_name no)
@@
 			(project "power v2"
 				(path "/7765ea03-990c-41e2-8b83-b7e84578cc41/8a309907-db9d-4e2b-b4b7-665a29344a77"
-					(reference "R6")
+					(reference "R8")
 					(unit 1)
 				)
@@
 		(dnp no)
 		(fields_autoplaced yes)
-		(property "Reference" "J2"
+		(property "Reference" "J4"
 			(at 50.8 34.29 0)
 			(show_name no)
@@
 			(project "power v2"
 				(path "/7765ea03-990c-41e2-8b83-b7e84578cc41/8a309907-db9d-4e2b-b4b7-665a29344a77"
-					(reference "J2")
+					(reference "J4")
 					(unit 1)
 				)
@@
 		(dnp no)
 		(fields_autoplaced yes)
-		(property "Reference" "#PWR016"
+		(property "Reference" "#PWR021"
 			(at 96.52 107.95 0)
 			(hide yes)
@@
 			(project "power v2"
 				(path "/7765ea03-990c-41e2-8b83-b7e84578cc41/8a309907-db9d-4e2b-b4b7-665a29344a77"
-					(reference "#PWR016")
+					(reference "#PWR021")
 					(unit 1)
 				)
@@
 		(dnp no)
 		(fields_autoplaced yes)
-		(property "Reference" "#PWR018"
+		(property "Reference" "#PWR020"
 			(at 90.17 68.58 0)
 			(hide yes)
@@
 			(project "power v2"
 				(path "/7765ea03-990c-41e2-8b83-b7e84578cc41/8a309907-db9d-4e2b-b4b7-665a29344a77"
-					(reference "#PWR018")
+					(reference "#PWR020")
 					(unit 1)
 				)
@@
 		(dnp no)
 		(fields_autoplaced yes)
-		(property "Reference" "#PWR011"
+		(property "Reference" "#PWR017"
 			(at 40.64 107.95 0)
 			(hide yes)
@@
 			(project "power v2"
 				(path "/7765ea03-990c-41e2-8b83-b7e84578cc41/8a309907-db9d-4e2b-b4b7-665a29344a77"
-					(reference "#PWR011")
+					(reference "#PWR017")
 					(unit 1)
 				)
@@
 		(dnp no)
 		(fields_autoplaced yes)
-		(property "Reference" "#PWR015"
+		(property "Reference" "#PWR019"
 			(at 50.8 86.36 0)
 			(hide yes)
@@
 			(project "power v2"
 				(path "/7765ea03-990c-41e2-8b83-b7e84578cc41/8a309907-db9d-4e2b-b4b7-665a29344a77"
-					(reference "#PWR015")
+					(reference "#PWR019")
 					(unit 1)
 				)
@@
 		(dnp no)
 		(fields_autoplaced yes)
-		(property "Reference" "R1"
+		(property "Reference" "R5"
 			(at 87.63 35.56 90)
 			(show_name no)
@@
 			(project "power v2"
 				(path "/7765ea03-990c-41e2-8b83-b7e84578cc41/8a309907-db9d-4e2b-b4b7-665a29344a77"
-					(reference "R1")
+					(reference "R5")
 					(unit 1)
 				)
@@
 		(dnp no)
 		(fields_autoplaced yes)
-		(property "Reference" "#PWR017"
+		(property "Reference" "#PWR022"
 			(at 106.68 68.58 0)
 			(hide yes)
@@
 			(project "power v2"
 				(path "/7765ea03-990c-41e2-8b83-b7e84578cc41/8a309907-db9d-4e2b-b4b7-665a29344a77"
-					(reference "#PWR017")
+					(reference "#PWR022")
 					(unit 1)
 				)
@@
 		(dnp no)
 		(fields_autoplaced yes)
-		(property "Reference" "D1"
+		(property "Reference" "D4"
 			(at 140.97 48.1964 90)
 			(show_name no)
@@
 			(project "power v2"
 				(path "/7765ea03-990c-41e2-8b83-b7e84578cc41/8a309907-db9d-4e2b-b4b7-665a29344a77"
-					(reference "D1")
+					(reference "D4")
 					(unit 1)
 				)
@@
 		(dnp no)
 		(fields_autoplaced yes)
-		(property "Reference" "#PWR019"
+		(property "Reference" "#PWR023"
 			(at 110.49 107.95 0)
 			(hide yes)
@@
 			(project "power v2"
 				(path "/7765ea03-990c-41e2-8b83-b7e84578cc41/8a309907-db9d-4e2b-b4b7-665a29344a77"
-					(reference "#PWR019")
-					(unit 1)
-				)
+					(reference "#PWR023")
+					(unit 1)
+				)
