File: hardware/pcb/prototypes/power-panel/v1/power-panel.kicad_pcb (KiCad board)
At the start: 2 copper layers, 18 parts, among them J1 Conn_01x09_Pin, J10 Conn_01x02_Pin, J11 Conn_01x03_Pin, J2 Conn_01x05_Pin, J3 Conn_01x03_Pin, J4 Conn_01x02_Pin, J5 Conn_01x02_Pin, J6 Conn_01x02_Pin, J7 Conn_01x07_Pin, J8 Conn_01x02_Pin, J9 Conn_01x05_Pin

Commit message: board layout
Parts:
- moved C7 164.5 mm to (184.2, 114.9), turned to 90 degrees
- moved J1 162.5 mm to (188.0, 56.5)
- moved C5 160.4 mm to (184.2, 97.8), turned to 90 degrees
- moved J3 158.9 mm to (188.0, 111.1)
- moved C6 157.8 mm to (184.2, 92.7), turned to 90 degrees
- moved C1 157.2 mm to (184.2, 75.6), turned to 90 degrees
- moved J2 156.1 mm to (188.0, 88.9)
- moved C2 155.2 mm to (184.2, 70.5), turned to 90 degrees
- moved C3 153.5 mm to (184.2, 65.4), turned to 90 degrees
- moved C4 152.3 mm to (184.2, 60.3), turned to 90 degrees
- moved J11 145.6 mm to (177.8, 111.1)
- moved J9 142.4 mm to (177.8, 88.9)
- moved J7 142.0 mm to (177.8, 56.5)
- moved J10 112.1 mm to (121.9, 112.4)
- moved J8 100.9 mm to (121.9, 92.7)
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Routing:
- net +5V: track 0.00 -> 62.9 mm

Commit message: board layout
Parts:
- C1, C2, C3, C4, C5, C6, C7: moved to B.Cu
- moved J1 48.3 mm to (139.7, 55.9)
- moved J3 48.3 mm to (139.7, 111.8)
- moved J2 48.3 mm to (139.7, 88.9)
- moved J7 43.3 mm to (134.6, 59.1)
- moved J11 43.2 mm to (134.6, 111.1)
- moved J9 43.2 mm to (134.6, 88.9)
- moved C1 40.7 mm to (143.5, 73.7), turned to 180 degrees
- moved C2 40.7 mm to (143.5, 68.6), turned to 180 degrees
- moved C3 40.7 mm to (143.5, 63.5), turned to 180 degrees
- moved C4 40.7 mm to (143.5, 58.4), turned to 180 degrees
- moved C5 40.7 mm to (143.5, 96.5), turned to 180 degrees
- moved C6 40.7 mm to (143.5, 91.4), turned to 180 degrees
- moved C7 40.6 mm to (143.5, 114.3), turned to 180 degrees
- moved J10 25.4 mm to (96.5, 112.4)
- moved J5 25.4 mm to (78.7, 85.1)
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Routing:
- net +5V: track 62.9 -> 115.8 mm
- net +3V3: track 0.00 -> 9.44 mm
- net +1V8: track 0.00 -> 9.44 mm
- net +0V9: track 0.00 -> 9.44 mm
- net +48V: track 0.00 -> 8.12 mm
- net +15V: track 0.00 -> 8.09 mm
- net -15V: track 0.00 -> 7.85 mm
- net GND: vias 0 -> 32
- added copper zone on B.Cu, net GND
- added copper zone on F.Cu, net GND
Other:
- board outline added: 71.1 x 73.7 mm
- board text added: "+15"
- board text added: "-15"
- board text added: "0V9"
- board text added: "1V8"
- board text added: "3V3"
- board text added: "48V"
- board text added: "5V"
- board text added: "Analog rails +15V -15V"
- board text added: "GND"
- board text added: "Low voltage +0.9V +1.8V +3.3V"
- board text added: "OpenMic Power board v0.2 (Power panel) 7/7/26"
- board text added: "Phantom power +48V"
- board text added: "USB supply +5V"
