File: hardware/pcb/prototypes/power/v2-5v/power v2.kicad_pcb (KiCad board)
At the start: 2 copper layers, 15.2 x 71.1 mm, 49 parts, among them J1 5V OUT, J2 USB_PD, J3 D_PIN, J4 USB_C_Receptacle_USB2.0_16P, J5 D_PIN, J6 GND, U1 TPS25730AD, U2 TUSB321, U3 TPS2116DRL

Commit message: board layout
Other:
- board text added: "OpenMic Power board v0.2 (5V only) 7/7/26"
- board text removed: "OpenMic Power board v0.2 (5V only) 7/4/26"
Changed lines of the file:
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@@
 			(at 3.175 0 0)
 			(layer "F.Fab")
+			(hide yes)
 			(effects
 				(font
@@
 		)
 	)
-	(gr_text "OpenMic\nPower board v0.2\n(5V only)\n7/4/26"
+	(gr_text "OpenMic\nPower board v0.2\n(5V only)\n7/7/26"
 		(at 91.44 63.5 90)
 		(layer "B.SilkS")
@@
 	)
 	(via
-		(at 86.36 52.07)
+		(at 86.36 51.562)
 		(size 0.6)
 		(drill 0.3)

Commit message: change to TPS25730AS
Parts:
- removed D2: R, LED_SMD:LED_0805_2012Metric_Pad1.15x1.40mm_HandSolder
- removed R4: 10k, Resistor_SMD:R_0805_2012Metric_Pad1.20x1.40mm_HandSolder
- removed TP1: VBUS_PD, TestPoint:TestPoint_Pad_1.5x1.5mm
- removed U1: TPS25730AD, Package_DFN_QFN:Texas_REF0038A_WQFN-38-2EP_6x4mm_P0.4
- added D5: R, LED_SMD:LED_0805_2012Metric_Pad1.15x1.40mm_HandSolder, F.Cu at (95.2, 83.2)
- added Q1: CSD87501L, openmic:BGA-10_P0.65mm, F.Cu at (90.2, 95.9)
- added R11: 4.7k, Resistor_SMD:R_0805_2012Metric_Pad1.20x1.40mm_HandSolder, F.Cu at (95.2, 85.7)
- added R12: 10k, Resistor_SMD:R_0805_2012Metric_Pad1.20x1.40mm_HandSolder, F.Cu at (95.2, 88.3)
- added TP5: VBUS_PD, TestPoint:TestPoint_Pad_1.5x1.5mm, F.Cu at (89.0, 83.8)
- added TP6: VSYS_PD, TestPoint:TestPoint_Pad_1.5x1.5mm, F.Cu at (91.5, 83.8)
- added U4: TPS25730AS, Package_DFN_QFN:VQFN-32-1EP_4x4mm_P0.4mm_EP2.8x2.8mm, F.Cu at (90.2, 90.8)
- moved C10 0.64 mm to (85.1, 90.8)
- moved C11 0.64 mm to (85.1, 93.3)
- moved C12 0.64 mm to (85.1, 95.9)
- moved C6 0.64 mm to (95.2, 95.9)
- moved C7 0.64 mm to (95.2, 93.3)
- moved C8 0.64 mm to (95.2, 90.8)
- moved C9 0.64 mm to (85.1, 88.3)
- moved R3 0.64 mm to (85.1, 83.2)
- moved R2 0.63 mm to (85.1, 85.7)
Connections:
- C10 pad 1: /5V PD/PPHV -> /5V PD/VSYS
- C11 pad 1: /5V PD/PPHV -> /5V PD/VSYS
- C12 pad 1: /5V PD/PPHV -> /5V PD/VSYS
- C20 pad 1: /5V PD/VBUS_PD -> /5V PD/VSYS
- R9 pad 1: /5V PD/VBUS_PD -> /5V PD/VSYS
- U3 pad 3: /5V PD/VBUS_PD -> /5V PD/VSYS
- U3 pad 5: /5V PD/VBUS_PD -> /5V PD/VSYS
Routing:
- net /5V PD/VSYS: track 0.00 -> 38.7 mm, vias 0 -> 2
- net /5V PD/VBUS_PD: track 65.2 -> 44.8 mm, vias 3 -> 2
- net Net-(U4-~{FAULT_IN}): track 0.00 -> 10.6 mm, vias 0 -> 2
- net Net-(D2-A): track 10.3 -> 0.00 mm, vias 2 -> 0
- net Net-(D5-A): track 0.00 -> 10.1 mm
- net /5V PD/PPHV: track 8.56 -> 0.00 mm
- net /5V PD/GATE_VBUS: track 0.00 -> 7.53 mm, vias 0 -> 2
- net /5V PD/CC1_PD: track 11.8 -> 18.1 mm, vias 2 -> 3
- net GND: track 41.4 -> 35.5 mm, vias 60 -> 75
- net /5V PD/LDO_3V3: track 22.7 -> 27.4 mm, vias 2 -> 4
- net Net-(U1-DRAIN-Pad15): track 4.48 -> 0.00 mm
- net /5V PD/CC2_PD: track 11.9 -> 14.8 mm, vias 2 -> 3
- net /5V PD/GATE_VSYS: track 0.00 -> 2.85 mm
- net /5V PD/ADCIN3: track 10.0 -> 11.7 mm
- net /5V PD/LDO_1V5: track 8.62 -> 10.3 mm, vias 0 -> 3
Other:
- board text added: "VSYS"
