File: hardware/pcb/prototypes/power/v2-5v/pd.kicad_sch (KiCad schematic)
At the start: 20 parts, among them J2 USB_PD, J3 D_PIN, U1 TPS25730AD

Commit message: change to TPS25730AS
Parts:
- removed D2: R, LED_SMD:LED_0805_2012Metric_Pad1.15x1.40mm_HandSolder, symbol Device:LED_Small
- removed R4: 10k, Resistor_SMD:R_0805_2012Metric_Pad1.20x1.40mm_HandSolder, symbol Device:R_US
- removed TP1: VBUS_PD, TestPoint:TestPoint_Pad_1.5x1.5mm, symbol Connector:TestPoint
- removed U1: TPS25730AD, Package_DFN_QFN:Texas_REF0038A_WQFN-38-2EP_6x4mm_P0.4, symbol openmic:TPS25730AD
- added D5: R, LED_SMD:LED_0805_2012Metric_Pad1.15x1.40mm_HandSolder, symbol Device:LED_Small
- added Q1: CSD87501L, openmic:BGA-10_P0.65mm, symbol openmic:CSD87501L
- added R11: 4.7k, Resistor_SMD:R_0805_2012Metric_Pad1.20x1.40mm_HandSolder, symbol Device:R_US
- added R12: 10k, Resistor_SMD:R_0805_2012Metric_Pad1.20x1.40mm_HandSolder, symbol Device:R_US
- added TP5: VBUS_PD, TestPoint:TestPoint_Pad_1.5x1.5mm, symbol Connector:TestPoint
- added TP6: VSYS_PD, TestPoint:TestPoint_Pad_1.5x1.5mm, symbol Connector:TestPoint
- added U4: TPS25730AS, Package_DFN_QFN:VQFN-32-1EP_4x4mm_P0.4mm_EP2.8x2.8mm, symbol openmic:TPS25730AS
Connections:
- net ADCIN3: now also U4.5 (ADCIN3)
- net CC1_PD: now also U4.24 (CC1)
- net CC2_PD: now also U4.25 (CC2)
- net GND: now also D5.1 (K), U4.11 (GND), U4.12 (GND), U4.14 (GND), U4.15 (GND), U4.16 (GND), U4.2 (ADCIN1), U4.22 (RESERVED), U4.28 (GND), U4.29 (GND), U4.3 (ADCIN2), U4.30 (RESERVED), U4.32 (VIN_3V3), U4.33 (GND), U4.8 (I2Ct_SDA), U4.9 (I2Ct_SCL)
- net LDO_1V5: now also U4.4 (LDO_1V5), U4.7 (ADCIN4)
- net LDO_3V3: now also R11.2, R12.2, U4.1 (LDO_3V3), U4.23 (PD5VMAX)
- net VBUS_PD: now also Q1.A2 (Source_2), Q1.B2 (Source_1), Q1.D2 (Source_1), Q1.E2 (Source_1), TP5.1, U4.26 (VBUS), U4.27 (VBUS)
- net PPHV renamed PD_OUT
- net PD_OUT: now also Q1.A1 (Source_1), Q1.B1 (Source_1), Q1.D1 (Source_1), Q1.E1 (Source_1), TP6.1, U4.19 (VSYS)
- new net: D5.2 (A), R11.1, U4.6 (CAP_MIS)
- new net: R12.1, U4.17 (~{FAULT_IN})
- new net GATE_VBUS: Q1.C2 (Gate_2), U4.21 (GATE_VBUS)
- new net GATE_VSYS: Q1.C1 (Gate_1), U4.20 (GATE_VSYS)
Other:
- moved on the sheet: C1, C10, C11, C12, C2, C3, C4, C5, C6, C7, C8, C9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

Commit message: update BOM
Parts:
- C1, C10, C11, C12, C2, C3, C4, C5, C6, C7, C8, C9: Type (none) -> Ceramic; Voltage (none) -> 10
