File: hardware/pcb/prototypes/power/v2-5v/power v2.kicad_sch (KiCad schematic)
At the start: 4 parts, among them J1 5V OUT, J6 GND

Commit message: change to TPS25730AS
Other:
- sheet 5V PD ports: added PD_OUT; removed VBUS_PD
- sheet Input Selector ports: added IN_PD, IN_USB; removed VBUS_PD, VBUS_USB
Changed lines of the file:
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@@
+			)
+		)
+		(property "MPN" ""
+			(at 147.32 64.77 90)
+			(hide yes)
+			(show_name no)
+			(do_not_autoplace no)
+			(effects
+				(font
+					(size 1.27 1.27)
+				)
 			)
 		)
@@
 			)
 		)
+		(property "MPN" ""
+			(at 142.24 78.74 0)
+			(hide yes)
+			(show_name no)
+			(do_not_autoplace no)
+			(effects
+				(font
+					(size 1.27 1.27)
+				)
+			)
+		)
 		(pin "2"
 		)
@@
 		)
 		(property "Description" "Generic connector, single row, 01x02, script generated"
+			(at 142.24 72.39 0)
+			(hide yes)
+			(show_name no)
+			(do_not_autoplace no)
+			(effects
+				(font
+					(size 1.27 1.27)
+				)
+			)
+		)
+		(property "MPN" ""
 			(at 142.24 72.39 0)
 			(hide yes)
@@
 			)
 		)
+		(property "MPN" ""
+			(at 139.7 64.77 0)
+			(hide yes)
+			(show_name no)
+			(do_not_autoplace no)
+			(effects
+				(font
+					(size 1.27 1.27)
+				)
+			)
+		)
 		(pin "1"
 		)
@@
 			)
 		)
-		(pin "VBUS_PD" input
-			(at 102.87 69.85 180)
-			(effects
-				(font
-					(size 1.27 1.27)
-				)
-				(justify left)
-			)
-		)
-		(pin "VBUS_USB" input
-			(at 102.87 76.2 180)
-			(effects
-				(font
-					(size 1.27 1.27)
-				)
-				(justify left)
-			)
-		)
 		(pin "VOUT" output
 			(at 129.54 69.85 0)
@@
 				)
 				(justify right)
+			)
+		)
+		(pin "IN_PD" input
+			(at 102.87 69.85 180)
+			(effects
+				(font
+					(size 1.27 1.27)
+				)
+				(justify left)
+			)
+		)
+		(pin "IN_USB" input
+			(at 102.87 76.2 180)
+			(effects
+				(font
+					(size 1.27 1.27)
+				)
+				(justify left)
 			)
 		)
@@
 			)
 		)
-		(pin "VBUS_PD" output
+		(pin "PD_OUT" output
 			(at 81.28 50.8 0)
 			(effects
