File: hardware/pcb/prototypes/power/v2-3v/low-voltage.kicad_pcb (KiCad board)
At the start: 2 copper layers, 43.2 x 31.8 mm, 23 parts, among them J3 Conn_01x02_Pin, J4 Conn_01x07_Pin, U1 TPS62172DSG, U2 TPS62171DSG, U5 TPS7A2009

Commit message: pcb layout
Parts:
- moved U1 0.40 mm to (113.7, 76.8)
- moved L2 0.40 mm to (113.7, 72.4)
- moved C2 0.40 mm to (110.5, 76.8)
- moved C6 0.40 mm to (116.8, 76.8)
- moved JP1 0.40 mm to (105.4, 74.7)
- moved R1 0.40 mm to (110.5, 72.4)
- moved R5 0.40 mm to (116.8, 72.4)
- moved L3 0.32 mm to (113.7, 62.2)
- moved U2 0.32 mm to (113.7, 66.7)
- moved C11 0.31 mm to (110.5, 54.0)
- moved C14 0.31 mm to (118.1, 54.0)
- moved C3 0.31 mm to (110.5, 66.7)
- moved C7 0.31 mm to (116.8, 66.7)
- moved JP2 0.31 mm to (105.4, 64.8)
- moved JP3 0.31 mm to (105.4, 54.6)
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Routing:
- net +1V8: track 0.00 -> 51.7 mm
- net +3V3: track 0.00 -> 37.5 mm
- net +5V: track 0.00 -> 34.5 mm
- net +0V9: track 0.00 -> 24.6 mm
- net Net-(JP2-B): track 0.00 -> 10.4 mm, vias 0 -> 2
- net Net-(JP1-B): track 0.00 -> 10.3 mm, vias 0 -> 2
- net Net-(JP3-B): track 0.00 -> 9.97 mm, vias 0 -> 2
- net Net-(U2-PG): track 0.00 -> 7.65 mm, vias 0 -> 2
- net Net-(U1-PG): track 0.00 -> 7.64 mm, vias 0 -> 2
- net Net-(U1-SW): track 0.00 -> 6.89 mm, vias 0 -> 2
- net Net-(U2-SW): track 0.00 -> 6.88 mm, vias 0 -> 2
- net Net-(D1-K): track 0.00 -> 2.57 mm
- net GND: vias 0 -> 44
- added copper zone on B.Cu, net GND
- added copper zone on F.Cu, net GND
Other:
- board text added: "+3V3"
- board text added: "EN 0V9"
- board text added: "EN 1V8"
- board text added: "EN 3V3"
- board text added: "OpenMic Power board v0.2 (15V only) 7/7/26"
- board text added: "TPS62171"
- board text added: "TPS62172"

Commit message: fix label
Other:
- board text added: "OpenMic Power board v0.2 (Low voltage) 7/8/26"
- board text removed: "OpenMic Power board v0.2 (15V only) 7/7/26"
Changed lines of the file:
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@@
 		)
 	)
-	(gr_text "OpenMic\nPower board v0.2\n(15V only)\n7/7/26"
+	(gr_text "OpenMic\nPower board v0.2\n(Low voltage)\n7/8/26"
 		(at 135.255 56.515 0)
 		(layer "B.SilkS")
