File: hardware/pcb/prototypes/power/v2-3v/low-voltage.kicad_sch (KiCad schematic)
At the start: 23 parts, among them J3 Conn_01x02_Pin, J4 Conn_01x07_Pin, U1 TPS62172DSG, U2 TPS62171DSG, U5 TPS7A2009

Commit message: update BOM
Parts:
- C11, C14: MPN CL21B105KBFNNNE -> (none); Type (none) -> Ceramic; Voltage (none) -> 6
- C2, C3: MPN CL21A106KAYNNNE -> (none); Type (none) -> Ceramic; Voltage (none) -> 10
- C6: MPN CL21A226MAQNNNE -> (none); Type (none) -> Ceramic; Voltage (none) -> 10
- C7: MPN CL21A226MAQNNNE -> (none); Type (none) -> Ceramic; Voltage (none) -> 6
- L2, L3: MPN ANR3015T2R2M -> (none)
- R1, R2, R5, R6, R7, R9: MPN 0805W8F1003T5E -> (none)
