File: hardware/pcb/prototypes/input/v2-inst/v2-inst/v2-inst.kicad_sch (KiCad schematic)
At the start: 57 parts, among them J1 TRS, J10 Conn_01x02_Pin, J11 XLR, J2 Conn_01x02_Pin, J3 Conn_01x03_Pin, J4 Conn_01x05_Pin, J5 Conn_01x09_Pin, J6 PH_EN, J7 Conn_01x06_Pin, J8 Conn_01x08_Pin, J9 OUT_BIAS, U1 THAT5263, U2 THAT1580, U3 OPA1637

Commit message: pcb layout
Parts:
- removed C10: 1000uF, Capacitor_THT:CP_Radial_D8.0mm_P3.50mm, symbol Device:C_Polarized_US
- removed C12, C13, C16, C17, C18: 100nF, Capacitor_SMD:C_0805_2012Metric_Pad1.18x1.45mm_HandSolder, symbol Device:C
- removed C19, C20: 10uF, Capacitor_THT:C_Radial_D5.0mm_H11.0mm_P2.00mm, symbol Device:C_Polarized_US
- removed C2, C3: 22pF, Capacitor_SMD:C_0805_2012Metric_Pad1.18x1.45mm_HandSolder, symbol Device:C
- removed C4: 220pF, Capacitor_SMD:C_0805_2012Metric_Pad1.18x1.45mm_HandSolder, symbol Device:C
- removed C5, C6: 47uF, Capacitor_THT:C_Radial_D10.0mm_H12.5mm_P5.00mm, symbol Device:C_Polarized_US
- removed C7: 100pF, Capacitor_SMD:C_0805_2012Metric_Pad1.18x1.45mm_HandSolder, symbol Device:C
- removed D4, D5, D6, D7: VTVS14ASMF, Diode_SMD:D_SMF, symbol Device:D_Zener
- removed J1: TRS, Connector_PinHeader_2.54mm:PinHeader_1x06_P2.54mm_Vertical, symbol Connector:Conn_01x06_Pin
- removed J10, J2: Conn_01x02_Pin, Connector_PinHeader_2.54mm:PinHeader_1x02_P2.54mm_Vertical, symbol Connector:Conn_01x02_Pin
- removed J11: XLR, Connector_PinHeader_2.54mm:PinHeader_1x05_P2.54mm_Vertical, symbol Connector:Conn_01x05_Pin
- removed J3: Conn_01x03_Pin, Connector_PinHeader_2.54mm:PinHeader_1x03_P2.54mm_Vertical, symbol Connector:Conn_01x03_Pin
- removed J4: Conn_01x05_Pin, Connector_PinHeader_2.54mm:PinHeader_1x05_P2.54mm_Vertical, symbol Connector:Conn_01x05_Pin
- removed J5: Conn_01x09_Pin, Connector_PinHeader_2.54mm:PinHeader_1x09_P2.54mm_Vertical, symbol Connector:Conn_01x09_Pin
- removed J6: PH_EN, Connector_PinHeader_2.54mm:PinHeader_1x02_P2.54mm_Vertical, symbol Connector:Conn_01x02_Pin
- removed J7: Conn_01x06_Pin, Connector_PinHeader_2.54mm:PinHeader_1x06_P2.54mm_Vertical, symbol Connector:Conn_01x06_Pin
- removed J8: Conn_01x08_Pin, Connector_PinHeader_2.54mm:PinHeader_1x08_P2.54mm_Vertical, symbol Connector:Conn_01x08_Pin
- removed R2, R3: 6k81, Resistor_SMD:R_0805_2012Metric_Pad1.20x1.40mm_HandSolder, symbol Device:R_US
- removed R4: 10, Resistor_SMD:R_0805_2012Metric_Pad1.20x1.40mm_HandSolder, symbol Device:R_US
- removed U1: THAT5263, Package_DFN_QFN:QFN-24-1EP_5x5mm_P0.65mm_EP3.4x3.4mm, symbol Audio:THAT5263
- removed U2: THAT1580, Package_DFN_QFN:QFN-16-1EP_4x4mm_P0.65mm_EP2.1x2.1mm_ThermalVias, symbol Audio:THAT1580
- added C10: 100nF, Capacitor_SMD:C_0805_2012Metric_Pad1.18x1.45mm_HandSolder, symbol Device:C
- added C12, C13: 10uF, Capacitor_THT:C_Radial_D5.0mm_H11.0mm_P2.00mm, symbol Device:C_Polarized_US
- added J1: PH, Connector_PinHeader_2.54mm:PinHeader_1x03_P2.54mm_Vertical, symbol Connector:Conn_01x03_Pin
- added J2: ANLG, Connector_PinHeader_2.54mm:PinHeader_1x05_P2.54mm_Vertical, symbol Connector:Conn_01x05_Pin
- added J3: LOWV, Connector_PinHeader_2.54mm:PinHeader_1x09_P2.54mm_Vertical, symbol Connector:Conn_01x09_Pin
- added J4: GND, Connector_PinHeader_2.54mm:PinHeader_1x02_P2.54mm_Vertical, symbol Connector:Conn_01x02_Pin
- added J5: TRS, Connector_PinHeader_2.54mm:PinHeader_1x06_P2.54mm_Vertical, symbol Connector:Conn_01x06_Pin
- added J6: XLR, Connector_PinHeader_2.54mm:PinHeader_1x05_P2.54mm_Vertical, symbol Connector:Conn_01x05_Pin
- added J7: SW CTRL, Connector_PinHeader_2.54mm:PinHeader_1x04_P2.54mm_Vertical, symbol Connector:Conn_01x04_Pin
- added J8: OUT_BIAS, Connector_PinHeader_2.54mm:PinHeader_1x02_P2.54mm_Vertical, symbol Connector:Conn_01x02_Pin
- added R18, R19: 10, Resistor_SMD:R_0805_2012Metric_Pad1.20x1.40mm_HandSolder, symbol Device:R_US
- added R20, R21: 5k, Resistor_SMD:R_0805_2012Metric_Pad1.20x1.40mm_HandSolder, symbol Device:R_US
- added SW1: DG1412EEQ, Package_SO:TSSOP-16_4.4x5mm_P0.65mm, symbol openmic:DG1412_TSSOP
- added U1: OPA1641, symbol Amplifier_Operational:OPA1641
- added U2: OPA1612AxD, Package_SO:SOIC-8_3.9x4.9mm_P1.27mm, symbol Amplifier_Operational:OPA1612AxD
- C14, C15: Voltage 6 -> 50
- C8: value 100pF -> 100nF; Type Film -> Ceramic
- C9: value 220pF -> 100nF; Type Film -> Ceramic
- J9: value OUT_BIAS -> OUT
- R10: value 2k -> 1k2
- R11, R12: value 2k -> 1k
- R14, R15: value 10 -> 2k
- R16, R17: value 5k -> 2k
- R5: value 10 -> 1k2
- R6, R7: value 1k2 -> 510
- R8: value 1M -> 510
- R9: value 2k -> 510
Connections:
- net +0V9: now also J3.2 (Pin_2)
- net +15V: now also C8.2, C10.1, J2.2 (Pin_2), SW1.13 (V+), U2.8 (V+); no longer C11.1, C15.1
- net +1V8: now also J3.4 (Pin_4)
- net +3V3: now also J3.6 (Pin_6)
- net +48V: now also J1.2 (Pin_2)
- net +5V: now also J3.8 (Pin_8)
- net -15V: now also C11.1, C15.1, C9.2, J2.4 (Pin_4), SW1.4 (V-), U2.4 (V-); no longer C15.2
- net Earth: now also C15.2, C9.1, C10.2, J1.1 (Pin_1), J1.3 (Pin_3), J2.1 (Pin_1), J2.3 (Pin_3), J2.5 (Pin_5), J3.1 (Pin_1), J3.3 (Pin_3), J3.5 (Pin_5), J3.7 (Pin_7), J3.9 (Pin_9), J4.1 (Pin_1), J4.2 (Pin_2), J5.1 (Pin_1), J5.4 (Pin_4), J5.6 (Pin_6), J6.1 (Pin_1), J6.4 (Pin_4), J6.5 (Pin_5), SW1.5 (GND), U2.3 (+), U2.6 (-); no longer R6.1, R7.2
- net at C1.1, D1.2 (A), R1.2: now also J5.2 (Pin_2)
- net at R13.1, U3.1 (VIN-): now also R15.2, R17.1; no longer R11.2, R9.1
- net at R5.1: now also R6.2, SW1.14 (S2), SW1.2 (D1)
- net at R16.2: now also U3.5 (VOUT-), R18.1
- net at R14.2: now also R13.2, R16.1, U3.8 (VIN+)
- net at R17.2: now also U3.4 (VOUT+), R19.1
- net at R8.1: now also R9.2, SW1.11 (S3)
- net at R8.2: now also R7.1, U2.2 (-)
- net at R11.1: now also R12.2, U2.5 (+)
- net at R10.1: now also R11.2, R15.1, SW1.7 (D4), U2.1
- new net: J7.1 (Pin_1), SW1.1 (IN1)
- new net: J7.2 (Pin_2), SW1.16 (IN2)
- new net: J7.4 (Pin_4), SW1.8 (IN4)
- new net: J7.3 (Pin_3), SW1.9 (IN3)
- new net: C12.2, R18.2
- new net: R10.2, R9.1, SW1.10 (D3), SW1.6 (S4)
- new net: JP1.2 (C), R20.1, R21.1
- new net: J8.1 (Pin_1), J8.2 (Pin_2), JP1.3 (B)
- new net: R6.1, R7.2, SW1.15 (D2)
- new net: C13.2, R19.2
- new net: R5.2, SW1.3 (S1)
- new net: C13.1, J9.1 (Pin_1), R20.2
- new net: C12.1, J9.2 (Pin_2), R21.2
- new net: R12.1, R14.1, U2.7
- new net TRS_R: J5.3 (Pin_3)
- new net TRS_T: J5.5 (Pin_5)
