File: hardware/pcb/prototypes/input/v2-line/v2-line.kicad_pcb (KiCad board)
At the start: 2 copper layers, 66 x 38.1 mm, 51 parts, among them J1 PH, J2 ANLG, J3 LOWV, J4 GND, J5 TRS, J6 XLR, J7 SW CTRL (3V3), J8 OUT_BIAS, J9 OUT, SW1 DG1412EEQ, U1 INA1650, U2 OPA1612AxD, U3 OPA1637

Commit message: add decoupling caps to sw
Parts:
- added C14: 100nF, Capacitor_SMD:C_0805_2012Metric_Pad1.18x1.45mm_HandSolder, F.Cu at (94.6, 102.9)
- added C15: 100nF, Capacitor_SMD:C_0805_2012Metric_Pad1.18x1.45mm_HandSolder, F.Cu at (106.0, 105.4)
- J7: value SW CTRL (3V3) -> SW CTRL
- moved C4 2.81 mm to (87.4, 98.4)
- moved C5 2.81 mm to (84.8, 98.4)
- moved C6 2.81 mm to (92.4, 98.4)
- moved D2 2.81 mm to (79.1, 98.4)
- moved D3 2.81 mm to (88.6, 109.9)
- moved R2 2.81 mm to (82.3, 98.4)
- moved R3 2.81 mm to (85.5, 109.9)
- moved U1 2.81 mm to (88.6, 104.1)
- moved C2 2.81 mm to (80.0, 103.5)
- moved C3 2.81 mm to (80.0, 109.2)
- moved C7 2.81 mm to (89.9, 98.4)
- moved R4 2.81 mm to (91.8, 109.9)
- moved C12 1.91 mm to (129.3, 97.8)
- moved C13 1.91 mm to (129.3, 110.5)
- moved R18 1.91 mm to (128.3, 102.2)
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Connections:
- SW1 pad 5: unconnected-(SW1A-GND-Pad5) -> Earth
Routing:
- net +15V: track 100.7 -> 134.7 mm
- net -15V: track 104.5 -> 115.3 mm
- net +3V3: track 63.9 -> 67.9 mm, vias 1 -> 2
- net Net-(SW1D-D3): track 17.5 -> 14.2 mm, vias 2 -> 0
- net /TRS_T: track 25.4 -> 22.6 mm
- net Earth: track 3.13 -> 5.33 mm, vias 176 -> 105
- net Net-(J7-Pin_3): track 20.9 -> 23.0 mm
- net Net-(J7-Pin_2): track 14.5 -> 16.4 mm, vias 1 -> 2
- net /TRS_R: track 25.8 -> 24.1 mm
- net Net-(R12-Pad1): track 14.0 -> 12.3 mm
- net Net-(SW1B-D1): track 13.8 -> 12.1 mm
- net Net-(J9-Pin_1): track 15.2 -> 16.6 mm
- net Net-(J7-Pin_1): track 16.3 -> 15.5 mm, vias 2 -> 1
- net Net-(J7-Pin_4): track 20.3 -> 19.7 mm
- net Net-(U2A--): track 21.3 -> 22.0 mm, vias 0 -> 2
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
Commit message: add labels
Other:
- board text added: "+0V9"
- board text added: "+15V"
- board text added: "+1V8"
- board text added: "+3V3"
- board text added: "+48V"
- board text added: "+5V"
- board text added: "-15V"
- board text added: "OpenMic Line input v0.2 7/24/26"
Changed lines of the file:
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@@
 			(at 0 7.46 90)
 			(layer "F.Fab")
+			(hide yes)
 			(effects
 				(font
@@
 			(at 0 12.54 90)
 			(layer "F.Fab")
+			(hide yes)
 			(effects
 				(font
@@
 			(at 0 22.7 90)
 			(layer "F.Fab")
+			(hide yes)
 			(effects
 				(font
@@
 	)
 	(gr_rect
+		(start 67.31 88.265)
+		(end 97.31 95.765)
+		(stroke
+			(width 0.08382)
+			(type default)
+		)
+		(fill no)
+		(layer "B.SilkS")
+	)
+	(gr_rect
 		(start 66.04 83.82)
 		(end 132.08 121.92)
@@
 		)
 	)
+	(gr_text "GND"
+		(at 68.58 87.74 90)
+		(layer "F.SilkS")
+		(effects
+			(font
+				(size 1 1)
+				(thickness 0.15)
+			)
+			(justify right)
+		)
+	)
+	(gr_text "+48V"
+		(at 71.12 87.74 90)
+		(layer "F.SilkS")
+		(effects
+			(font
+				(size 1 1)
+				(thickness 0.15)
+			)
+			(justify right)
+		)
+	)
+	(gr_text "GND"
+		(at 73.66 87.74 90)
+		(layer "F.SilkS")
+		(effects
+			(font
+				(size 1 1)
+				(thickness 0.15)
+			)
+			(justify right)
+		)
+	)
+	(gr_text "GND"
+		(at 86.36 87.74 90)
+		(layer "F.SilkS")
+		(effects
+			(font
+				(size 1 1)
+				(thickness 0.15)
+			)
+			(justify right)
+		)
+	)
+	(gr_text "-15V"
+		(at 88.9 87.74 90)
+		(layer "F.SilkS")
+		(effects
+			(font
+				(size 1 1)
+				(thickness 0.15)
+			)
+			(justify right)
+		)
+	)
+	(gr_text "GND"
+		(at 91.44 87.74 90)
+		(layer "F.SilkS")
+		(effects
+			(font
+				(size 1 1)
+				(thickness 0.15)
+			)
+			(justify right)
+		)
+	)
+	(gr_text "+15V"
+		(at 93.98 87.74 90)
+		(layer "F.SilkS")
+		(effects
+			(font
+				(size 1 1)
+				(thickness 0.15)
+			)
+			(justify right)
+		)
+	)
+	(gr_text "GND"
+		(at 96.52 87.74 90)
+		(layer "F.SilkS")
+		(effects
+			(font
+				(size 1 1)
+				(thickness 0.15)
+			)
+			(justify right)
+		)
+	)
+	(gr_text "GND"
+		(at 109.22 87.74 90)
+		(layer "F.SilkS")
+		(effects
+			(font
+				(size 1 1)
+				(thickness 0.15)
+			)
+			(justify right)
+		)
+	)
+	(gr_text "+5V"
+		(at 111.76 87.74 90)
+		(layer "F.SilkS")
+		(effects
+			(font
+				(size 1 1)
+				(thickness 0.15)
+			)
+			(justify right)
+		)
+	)
+	(gr_text "GND"
+		(at 114.3 87.74 90)
+		(layer "F.SilkS")
+		(effects
+			(font
+				(size 1 1)
+				(thickness 0.15)
+			)
+			(justify right)
+		)
+	)
+	(gr_text "+3V3"
+		(at 116.84 87.74 90)
+		(layer "F.SilkS")
+		(effects
+			(font
+				(size 1 1)
+				(thickness 0.15)
+			)
+			(justify right)
+		)
+	)
+	(gr_text "GND"
+		(at 119.38 87.74 90)
+		(layer "F.SilkS")
+		(effects
+			(font
+				(size 1 1)
+				(thickness 0.15)
+			)
+			(justify right)
+		)
+	)
+	(gr_text "+1V8"
+		(at 121.92 87.74 90)
+		(layer "F.SilkS")
+		(effects
+			(font
+				(size 1 1)
+				(thickness 0.15)
+			)
+			(justify right)
+		)
+	)
+	(gr_text "GND"
+		(at 124.46 87.74 90)
+		(layer "F.SilkS")
+		(effects
+			(font
+				(size 1 1)
+				(thickness 0.15)
+			)
+			(justify right)
+		)
+	)
+	(gr_text "+0V9"
+		(at 127 87.74 90)
+		(layer "F.SilkS")
+		(effects
+			(font
+				(size 1 1)
+				(thickness 0.15)
+			)
+			(justify right)
+		)
+	)
+	(gr_text "GND"
+		(at 129.54 87.74 90)
+		(layer "F.SilkS")
+		(effects
+			(font
+				(size 1 1)
+				(thickness 0.15)
+			)
+			(justify right)
+		)
+	)
+	(gr_text "OpenMic\nLine input v0.2\n7/24/26"
+		(at 131.445 94.615 0)
+		(layer "B.SilkS")
+		(effects
+			(font
+				(size 1.5 1.5)
+				(thickness 0.3)
+				(bold yes)
+			)
+			(justify left bottom mirror)
+		)
+	)

Commit message: add RFI protection
Parts:
- removed R2, R3: 100k, Resistor_SMD:R_0805_2012Metric_Pad1.20x1.40mm_HandSolder
- added C16: 330pF, Capacitor_SMD:C_0805_2012Metric_Pad1.18x1.45mm_HandSolder, F.Cu at (80.6, 106.7)
- added C17: 330pF, Capacitor_SMD:C_0805_2012Metric_Pad1.18x1.45mm_HandSolder, F.Cu at (80.6, 111.8)
- added R22: 100, Resistor_SMD:R_0805_2012Metric_Pad1.20x1.40mm_HandSolder, F.Cu at (78.1, 111.8)
- added R23: 100, Resistor_SMD:R_0805_2012Metric_Pad1.20x1.40mm_HandSolder, F.Cu at (78.1, 106.7)
- moved R4 10.0 mm to (83.2, 104.8)
- moved C3 3.86 mm to (83.8, 109.9)
- moved D2 3.85 mm to (81.3, 95.2)
- moved C2 3.24 mm to (79.4, 100.3)
- moved D3 0.91 mm to (89.5, 109.9)
Connections:
- C2 pad 1: /TRS_T -> Net-(C17-Pad1)
- C3 pad 1: /TRS_R -> Net-(C16-Pad1)
- D2 pad 3: /TRS_T -> Net-(C17-Pad1)
- D3 pad 3: /TRS_R -> Net-(C16-Pad1)
Routing:
- net Net-(C17-Pad1): track 0.00 -> 18.0 mm, vias 0 -> 1
- net /TRS_R: track 24.1 -> 10.1 mm
- net /TRS_T: track 22.6 -> 10.2 mm
- net Net-(C16-Pad1): track 0.00 -> 8.08 mm
- net Net-(U1A-COM): track 8.30 -> 2.70 mm
- net +15V: track 134.7 -> 130.5 mm
- net -15V: track 115.3 -> 111.2 mm
- net Net-(U1A-IN+): track 4.03 -> 5.43 mm
- net Earth: vias 105 -> 110
