File: hardware/pcb/main-board/power.kicad_sch (KiCad schematic)
At the start: 64 parts, among them J9 USB_C_Receptacle_USB2.0_16P, SW16 SW_Push, T1 475uH, U20 TPS7A39, U21 SN6505BDBV, U22 TPS2116DRL, U23 TPS62172DSG, U25 TPS7A2009, U26 TPS62171DSG, U27 TPS7A4101, U28 TPS61391, U29 CH224K

Commit message: update power supply to prototype circuit
Parts:
- removed C163: 22uF, Capacitor_SMD:C_0805_2012Metric_Pad1.18x1.45mm_HandSolder, symbol Device:C
- removed C180: 1uF, Capacitor_SMD:C_0805_2012Metric_Pad1.18x1.45mm_HandSolder, symbol Device:C
- removed C198: 10uF, Capacitor_SMD:C_0805_2012Metric_Pad1.18x1.45mm_HandSolder, symbol Device:C_Small
- removed J9: USB_C_Receptacle_USB2.0_16P, Connector_USB:USB_C_Receptacle_HRO_TYPE-C-31-M-12, symbol Connector:USB_C_Receptacle_USB2.0_16P
- removed R110: 330k, Resistor_SMD:R_0805_2012Metric_Pad1.20x1.40mm_HandSolder, symbol Device:R_US
- removed R111: 100k, Resistor_SMD:R_0805_2012Metric_Pad1.20x1.40mm_HandSolder, symbol Device:R_US
- removed R113: 10k, Resistor_SMD:R_0603_1608Metric_Pad0.98x0.95mm_HandSolder, symbol Device:R_Small_US
- removed R122: 10k, Resistor_SMD:R_0805_2012Metric_Pad1.20x1.40mm_HandSolder, symbol Device:R_US
- removed U22: TPS2116DRL, Package_TO_SOT_SMD:SOT-583-8, symbol Power_Management:TPS2116DRL
- removed U29: CH224K, Package_SO:SSOP-10-1EP_3.9x4.9mm_P1mm_EP2.1x3.3mm, symbol Interface_USB:CH224K
- added C116, C117: 330pF, Capacitor_SMD:C_0805_2012Metric_Pad1.18x1.45mm_HandSolder, symbol Device:C_Small
- added C118, C151: 10uF, Capacitor_SMD:C_0805_2012Metric_Pad1.18x1.45mm_HandSolder, symbol Device:C_Small
- added C119, C73: 4.7uF, Capacitor_SMD:C_0805_2012Metric_Pad1.18x1.45mm_HandSolder, symbol Device:C_Small
- added C124, C150: 22uF, Capacitor_SMD:C_0805_2012Metric_Pad1.18x1.45mm_HandSolder, symbol Device:C_Small
- added C163, C180: 1uF, Capacitor_SMD:C_0805_2012Metric_Pad1.18x1.45mm_HandSolder, symbol Device:C_Small
- added C74, C77, C78, C79: 10nF, Capacitor_SMD:C_0805_2012Metric_Pad1.18x1.45mm_HandSolder, symbol Device:C_Small
- added J2: USB_PD, Connector_USB:USB_C_Receptacle_HRO_TYPE-C-31-M-12, symbol Connector:USB_C_Receptacle_USB2.0_16P
- added Q4: CSD87501L, openmic:BGA-10_P0.65mm, symbol openmic:CSD87501L
- added R110: 220k, Resistor_SMD:R_0805_2012Metric_Pad1.20x1.40mm_HandSolder, symbol Device:R_Small_US
- added R111: 68k, Resistor_SMD:R_0805_2012Metric_Pad1.20x1.40mm_HandSolder, symbol Device:R_Small_US
- added R143, R144: 200k, Resistor_SMD:R_0805_2012Metric_Pad1.20x1.40mm_HandSolder, symbol Device:R_US
- added R3: 180k, Resistor_SMD:R_0805_2012Metric_Pad1.20x1.40mm_HandSolder, symbol Device:R_Small_US
- added R46: 10k, Resistor_SMD:R_0805_2012Metric_Pad1.20x1.40mm_HandSolder, symbol Device:R_Small_US
- added R53: 10k, Resistor_SMD:R_0805_2012Metric_Pad1.20x1.40mm_HandSolder, symbol Device:R_US
- added R94: 4.7k, Resistor_SMD:R_0805_2012Metric_Pad1.20x1.40mm_HandSolder, symbol Device:R_US
- added U10: TPS25730AS, Package_DFN_QFN:VQFN-32-1EP_4x4mm_P0.4mm_EP2.8x2.8mm, symbol openmic:TPS25730AS
- added U18: TPS2116DRL, Package_TO_SOT_SMD:SOT-583-8, symbol Power_Management:TPS2116DRL
- C197: value 100nF -> 22uF; Type (none) -> Ceramic; Voltage (none) -> 10
- R103: value 118k -> 120k
- R109: value 127k -> 130k
- R115: value 475k -> 200k
- R118: value 392k -> 200k
- R119: value 12k -> 10k
Connections:
- net VBUS is gone; now on net +5V: C197.1
- net +5V: now also U18.2 (VOUT), U18.7 (VOUT)
- net +5V_USB: now also C180.1, U18.6 (VIN2)
- net Earth: now also C116.2, C117.2, C118.2, C119.2, C124.2, C150.2, C151.2, C163.2, C180.2, C73.2, C74.2, C77.2, C78.2, C79.2, J2.A1 (GND), J2.A12 (GND), J2.B1 (GND), J2.B12 (GND), J2.SH (SHIELD), R111.2, R46.2, U10.11 (GND), U10.12 (GND), U10.14 (GND), U10.15 (GND), U10.16 (GND), U10.2 (ADCIN1), U10.22 (RESERVED), U10.28 (GND), U10.29 (GND), U10.3 (ADCIN2), U10.30 (RESERVED), U10.32 (VIN_3V3), U10.33 (GND), U10.8 (I2Ct_SDA), U10.9 (I2Ct_SCL), U18.1 (GND)
- net PD_PWR_IND: now also R94.1, U10.6 (CAP_MIS)
- net at C172.1, C173.1, C174.1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: now also R143.1; no longer R118.1
- net at C176.2, R119.1, U27.2 (FB): now also R144.2; no longer R115.2
- new net: R53.1, U10.17 (~{FAULT_IN})
- new net: R118.1, R143.2
- new net: R115.2, R144.1
- new net: J2.A6 (D+), J2.B6 (D+)
- new net: J2.A7 (D-), J2.B7 (D-)
- new net ADCIN3: R3.2, R46.1, U10.5 (ADCIN3)
- new net CC1_PD: C116.1, J2.A5 (CC1), U10.24 (CC1)
- new net CC2_PD: C117.1, J2.B5 (CC2), U10.25 (CC2)
- new net GATE_VBUS: Q4.C2 (Gate_2), U10.21 (GATE_VBUS)
- new net GATE_VSYS: Q4.C1 (Gate_1), U10.20 (GATE_VSYS)
- new net LDO_1V5: C119.1, U10.4 (LDO_1V5), U10.7 (ADCIN4)
- new net LDO_3V3: C118.1, R3.1, R53.2, R94.2, U10.1 (LDO_3V3), U10.23 (PD5VMAX)
- new net PR1: R110.2, R111.1, U18.4 (PR1)
- new net VBUS_PD: C73.1, C74.1, C77.1, C78.1, C79.1, J2.A4 (VBUS), J2.A9 (VBUS), J2.B4 (VBUS), J2.B9 (VBUS), Q4.A2 (Source_2), Q4.B2 (Source_1), Q4.D2 (Source_1), Q4.E2 (Source_1), U10.26 (VBUS), U10.27 (VBUS)
- new net VSYS_PD: C124.1, C150.1, C151.1, C163.1, Q4.A1 (Source_1), Q4.B1 (Source_1), Q4.D1 (Source_1), Q4.E1 (Source_1), R110.1, U10.19 (VSYS), U18.3 (VIN1), U18.5 (MODE)
Other:
- note added: "ADCIN1 - 0 ADCIN2 - 0 ADCIN3 - 1 ADCIN4 - 5 Provides 5V at 1.5A operating current 3A max"
- note added: "CAP_MIS pulled low when source can't provide 1.5A LED is ON when source is OK"
- note added: "R_down / (R_down + R_up) ratio min target max 0.0229 0.0475 0.0722"
- moved on the sheet: R119

Commit message: add ptc fuses to phantom and usb supplies
Parts:
- added D70: LED, LED_SMD:LED_0603_1608Metric_Pad1.05x0.95mm_HandSolder, symbol Device:LED
- added F1: 40mA, symbol Device:Polyfuse
- added F2: 1.6A, symbol Device:Polyfuse
- added R122: 47k, Resistor_SMD:R_0805_2012Metric_Pad1.20x1.40mm_HandSolder, symbol Device:R_US
Connections:
- net +48V_PH: now also D70.1 (K), F1.2; no longer C176.1, C177.1, C178.1, R115.1, U27.1 (OUT)
- net VBUS_PD: now also F2.1; no longer J2.A4 (VBUS), J2.A9 (VBUS), J2.B4 (VBUS), J2.B9 (VBUS)
- new net: C176.1, C177.1, C178.1, F1.1, R115.1, R122.1, U27.1 (OUT)
- new net: D70.2 (A), R122.2
- new net: F2.2, J2.A4 (VBUS), J2.A9 (VBUS), J2.B4 (VBUS), J2.B9 (VBUS)
Other:
- note added: "LED indicates blown fuse"
