File: hardware/pcb/prototypes/input/v3/diff-driver.kicad_sch (KiCad schematic)
At the start: 16 parts, among them J5 OUT_BIAS, U3 OPA1637

Commit message: add ground pin to audio outputs
Parts:
- C21, C22: Type Electrolytic -> Bipolar Electrolytic
Changed lines of the file:
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@@
 			)
 		)
-		(property "Type" "Electrolytic"
+		(property "Type" "Bipolar Electrolytic"
 			(at 181.61 90.17 90)
 			(hide yes)
@@
 			)
 		)
-		(property "Type" "Electrolytic"
+		(property "Type" "Bipolar Electrolytic"
 			(at 181.61 95.25 90)
 			(hide yes)
