File: hardware/pcb/prototypes/input/v3/inst.kicad_sch (KiCad schematic)
At the start: 6 parts, among them U5 OPA1641

Commit message: add ground pin to audio outputs
Parts:
- C31: Type C0G/NP0 Ceramic -> C0G Ceramic
Changed lines of the file:
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@@
 			)
 		)
-		(property "Type" "C0G/NP0 Ceramic"
+		(property "Type" "C0G Ceramic"
 			(at 116.84 107.95 0)
 			(hide yes)
