File: hardware/pcb/prototypes/input/v3/line.kicad_sch (KiCad schematic)
At the start: 14 parts, among them U4 INA1650

Commit message: add ground pin to audio outputs
Parts:
- C23, C24: Type C0G/NP0 Ceramic -> C0G Ceramic
- C25, C26: Type Electrolytic -> Bipolar Electrolytic
Changed lines of the file:
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@@
 			)
 		)
-		(property "Type" "Electrolytic"
+		(property "Type" "Bipolar Electrolytic"
 			(at 128.27 101.6 90)
 			(hide yes)
@@
 			)
 		)
-		(property "Type" "C0G/NP0 Ceramic"
+		(property "Type" "C0G Ceramic"
 			(at 74.93 118.11 0)
 			(hide yes)
@@
 			)
 		)
-		(property "Type" "Electrolytic"
+		(property "Type" "Bipolar Electrolytic"
 			(at 128.27 111.76 90)
 			(hide yes)
@@
 			)
 		)
-		(property "Type" "C0G/NP0 Ceramic"
+		(property "Type" "C0G Ceramic"
 			(at 67.31 118.11 0)
 			(hide yes)
