File: hardware/pcb/prototypes/input/v3/mic.kicad_sch (KiCad schematic)
At the start: 30 parts, among them J3 PH_EN, J4 Conn_01x08_Pin, U1 THAT5263, U2 THAT1580

Commit message: add ground pin to audio outputs
Parts:
- C10, C11, C4, C5, C6, C9: Type Film -> C0G Ceramic
- C7, C8: Type Electrolytic -> Bipolar Electrolytic
Changed lines of the file:
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@@
 			)
 		)
-		(property "Type" "Film"
+		(property "Type" "C0G Ceramic"
 			(at 91.44 118.11 0)
 			(hide yes)
@@
 			)
 		)
-		(property "Type" "Film"
+		(property "Type" "C0G Ceramic"
 			(at 180.34 100.33 0)
 			(hide yes)
@@
 			)
 		)
-		(property "Type" "Film"
+		(property "Type" "C0G Ceramic"
 			(at 91.44 100.33 0)
 			(hide yes)
@@
 			)
 		)
-		(property "Type" "Film"
+		(property "Type" "C0G Ceramic"
 			(at 195.58 105.41 0)
 			(hide yes)
@@
 			)
 		)
-		(property "Type" "Electrolytic"
+		(property "Type" "Bipolar Electrolytic"
 			(at 134.62 114.3 90)
 			(hide yes)
@@
 			)
 		)
-		(property "Type" "Film"
+		(property "Type" "C0G Ceramic"
 			(at 180.34 110.49 0)
 			(hide yes)
@@
 			)
 		)
-		(property "Type" "Film"
+		(property "Type" "C0G Ceramic"
 			(at 104.14 105.41 0)
 			(hide yes)
@@
 			)
 		)
-		(property "Type" "Electrolytic"
+		(property "Type" "Bipolar Electrolytic"
 			(at 134.62 96.52 90)
 			(hide yes)
