File: hardware/pcb/prototypes/input/v3/v3.kicad_pcb (KiCad board)
At the start: 4 copper layers, 106.7 x 81.3 mm, 155 parts, among them J1 NMJ6HHD2, J10 LINE CTRL, J11 INST CTRL, J12 OUT_BIAS, J13 OUT_BIAS, J14 OUT_MIC, J15 OUT_LINE, J16 OUT_INST, J17 Conn_01x02_Pin, J2 NCJ10FI-H, J3 PH_EN, J4 Conn_01x08_Pin, J5 OUT_BIAS, J6 Conn_01x03_Pin, J7 Conn_01x05_Pin, J8 Conn_01x09_Pin, J9 Conn_01x02_Pin, SW1 DG1412EEQ, SW2 DG1412EEQ, U1 THAT5263, U2 THAT1580, U3 OPA1637, U4 INA1650, U5 OPA1641, U6 OPA1612AxD, U7 OPA1612AxD, U8 OPA1637, U9 OPA1637

Commit message: add ground pin to audio outputs
Parts:
- removed J14: OUT_MIC, Connector_PinHeader_2.54mm:PinHeader_1x02_P2.54mm_Vertical
- removed J15: OUT_LINE, Connector_PinHeader_2.54mm:PinHeader_1x02_P2.54mm_Vertical
- removed J16: OUT_INST, Connector_PinHeader_2.54mm:PinHeader_1x02_P2.54mm_Vertical
- added J18: OUT_MIC, Connector_PinHeader_2.54mm:PinHeader_1x03_P2.54mm_Vertical, F.Cu at (127.0, 27.9)
- added J19: OUT_LINE, Connector_PinHeader_2.54mm:PinHeader_1x03_P2.54mm_Vertical, F.Cu at (127.0, 50.8)
- added J20: OUT_INST, Connector_PinHeader_2.54mm:PinHeader_1x03_P2.54mm_Vertical, F.Cu at (127.0, 73.7)
- J10: value LINE CTRL -> SW CTRL
- J11: value INST CTRL -> SW CTRL
Routing:
- net /Diff Driver/DIFF_OUT_P: track 28.5 -> 32.4 mm
- net /Diff Driver2/DIFF_OUT_P: track 34.1 -> 37.8 mm
- net /Diff Driver1/DIFF_OUT_P: track 23.8 -> 27.0 mm
- net Earth: vias 150 -> 154
