File: hardware/pcb/prototypes/input/v3/v3.kicad_sch (KiCad schematic)
At the start: 14 parts, among them J1 NMJ6HHD2, J14 OUT_MIC, J15 OUT_LINE, J16 OUT_INST, J2 NCJ10FI-H

Commit message: add ground pin to audio outputs
Parts:
- removed J14: OUT_MIC, Connector_PinHeader_2.54mm:PinHeader_1x02_P2.54mm_Vertical, symbol Connector:Conn_01x02_Pin
- removed J15: OUT_LINE, Connector_PinHeader_2.54mm:PinHeader_1x02_P2.54mm_Vertical, symbol Connector:Conn_01x02_Pin
- removed J16: OUT_INST, Connector_PinHeader_2.54mm:PinHeader_1x02_P2.54mm_Vertical, symbol Connector:Conn_01x02_Pin
- added J18: OUT_MIC, Connector_PinHeader_2.54mm:PinHeader_1x03_P2.54mm_Vertical, symbol Connector:Conn_01x03_Pin
- added J19: OUT_LINE, Connector_PinHeader_2.54mm:PinHeader_1x03_P2.54mm_Vertical, symbol Connector:Conn_01x03_Pin
- added J20: OUT_INST, Connector_PinHeader_2.54mm:PinHeader_1x03_P2.54mm_Vertical, symbol Connector:Conn_01x03_Pin
Connections:
- net Diff Driver/DIFF_OUT_N: now also J18.3 (Pin_3)
- net Diff Driver/DIFF_OUT_P: now also J18.1 (Pin_1)
- net Diff Driver1/DIFF_OUT_N: now also J19.3 (Pin_3)
- net Diff Driver1/DIFF_OUT_P: now also J19.1 (Pin_1)
- net Diff Driver2/DIFF_OUT_N: now also J20.3 (Pin_3)
- net Diff Driver2/DIFF_OUT_P: now also J20.1 (Pin_1)
- net GNDA: now also J18.2 (Pin_2), J19.2 (Pin_2), J20.2 (Pin_2)
