File: hardware/pcb/prototypes/power/v2-15v/analog-rails.kicad_sch (KiCad schematic)
At the start: 30 parts, among them J1 Conn_01x02_Pin, J2 Conn_01x05_Pin, T1 475uH, U1 SN6505BDBV, U2 TPS7A39

Commit message: update BOM
Parts:
- C1, C5: Voltage (none) -> 10
- C2, C3, C4, C6, C7: Voltage (none) -> 50

Commit message: update resistor value
Parts:
- R2: value 470 -> 470k
Changed lines of the file:
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@@
 			)
 		)
-		(property "Value" "470"
+		(property "Value" "470k"
 			(at 156.21 60.9599 0)
 			(show_name no)
