File: hardware/pcb/prototypes/power/v2-15v/analog-rails.kicad_pcb (KiCad board)
At the start: 2 copper layers, 43.2 x 17.8 mm, 30 parts, among them J1 Conn_01x02_Pin, J2 Conn_01x05_Pin, T1 475uH, U1 SN6505BDBV, U2 TPS7A39

Commit message: update resistor value
Parts:
- R2: value 470 -> 470k
